Commit message: update

File: kubot_description/urdf/camera_xacro/non-3dsensor.urdf.xacro (robot description, xacro)
@@ -3,5 +3,5 @@
 <xacro:include filename="$(find kubot_description)/urdf/kubot_properties.urdf.xacro"/>
     <xacro:macro
-    name="sensor"
+    name="camera_sensor"
     params="frame:=camera_link camera_joint_xyz:=0 camera_joint_rpy:=0">
     </xacro:macro>

File: kubot_description/urdf/lidar_xacro/rplidar-a1.urdf.xacro (robot description, xacro)
@@ -10,5 +10,5 @@
       <origin xyz="0 0 -0.0241" rpy="0 0 3.1415"/>
       <geometry>
-        <mesh filename="package://kubot_description/meshes/lidar_frame/rplidar-a1/laser_link.stl" scale="0.001 0.001 0.001"/>
+        <mesh filename="package://kubot_description/meshes/lidar_frame/$(arg lidar)/laser_link.stl" scale="0.001 0.001 0.001"/>
       </geometry>
       <xacro:material_dark_grey/>

File: kubot_description/urdf/lidar_xacro/two-rplidar-a2.urdf.xacro (robot description, xacro)
@@ -1,64 +1,205 @@
 <?xml version="1.0"?>
-<robot name="kubot" xmlns:xacro="https://ros.org/wiki/xacro">
-  <xacro:include filename="$(find kubot_description)/urdf/kubot_properties.urdf.xacro"/>
-  <xacro:macro
-  name="lidar"
-  params="frame:=laser_link lidar_enabled:=true lidar_joint_xyz:=0 lidar_joint_rpy:=0 lidar1_joint_xyz:=0 lidar1_joint_rpy:=0 lidar2_joint_xyz:=0 lidar2_joint_rpy:=0">
-      <xacro:if value="${lidar_enabled}">
-        <link name="lidar">
-        </link>
-        <!-- laser 1  link -->
-        <link name="lidar1">
-            <visual>
-                <origin xyz="0 0 0.031" rpy="0 0 0"/>
-                <geometry>
-                    <mesh filename="package://kubot_description/meshes/lidar_frame/rplidar-a2/laser_link.stl" scale="0.001 0.001 0.001"/>
-                </geometry>
-            <xacro:material_dark_grey/>
-            </visual>
-            <collision>
-                <origin xyz="0 0 0.031" rpy="0 0 0"/>
-                <geometry>
-                    <mesh filename="package://kubot_description/meshes/lidar_frame/rplidar-a2/laser_link.stl" scale="0.001 0.001 0.001"/>
-                </geometry>
-            <xacro:material_white/>
-            </collision>
-        </link>
-        <!-- laser 2  link -->
-        <link name="lidar2">
-            <visual>
-                <origin xyz="0 0 0.031" rpy="0 0 0"/>
-                <geometry>
-                    <mesh filename="package://kubot_description/meshes/lidar_frame/rplidar-a2/laser_link.stl" scale="0.001 0.001 0.001"/>
-                </geometry>
-            <xacro:material_dark_grey/>
-            </visual>
-            <collision>
-                <origin xyz="0 0 0.031" rpy="0 0 0"/>
-                <geometry>
-                    <mesh filename="package://kubot_description/meshes/lidar_frame/rplidar-a2/laser_link.stl" scale="0.001 0.001 0.001"/>
-                </geometry>
-            <xacro:material_white/>
-            </collision>
-        </link>
-        <!-- lidar  joint -->
-        <joint name="lidar_joint" type="fixed">
-            <origin xyz="${lidar_joint_xyz}" rpy="${lidar_joint_rpy}" />
-            <parent link="base_link" />
-            <child link="lidar" />
-        </joint>
-        <!-- lidar  1 joint -->
-        <joint name="lidar1_joint" type="fixed">
-            <origin xyz="0.319 0.208 0.166" rpy="0 0 0.7854" />
-            <parent link="base_link" />
-            <child link="lidar1" />
-        </joint>
-        <!-- lidar  2 joint -->
-        <joint name="lidar2_joint" type="fixed">
-            <origin xyz="-0.319 -0.208 0.166" rpy="0 0 -2.355" />
-            <parent link="base_link" />
-            <child link="lidar2" />
-        </joint>
-      </xacro:if>
+<robot name="kubot_robot" xmlns:xacro="https://ros.org/wiki/xacro">
+<xacro:include filename="$(find kubot_description)/urdf/kubot_properties.urdf.xacro"/>
+<xacro:macro
+name="lidar"
+params="frame:=laser_link lidar_joint_xyz:=0 lidar_joint_rpy:=0">
+<!-- Laser Frame -->
+  <link name="${frame}">
+    <visual>
+        <origin xyz="0 0 0.031" rpy="0 0 0"/>
+        <geometry>
+            <mesh filename="package://kubot_description/meshes/lidar_frame/$(arg lidar)/laser_link.stl" scale="0.001 0.001 0.001"/>
+        </geometry>
+      <xacro:material_dark_grey/>
+    </visual>
+    <collision>
+        <origin xyz="0 0 0.031" rpy="0 0 0"/>
+        <geometry>
+            <cylinder length="0.0515" radius="0.055"/>
+        </geometry>
+        <xacro:material_white/>
+    </collision>
+    <inertial>
+      <origin xyz="0 0 -0.0241" rpy="0 0 3.1415"/>
+      <mass value="0.179"/>
+      <inertia
+        ixx="0.001"
+        ixy="0.0"
+        ixz="0.0"
+        iyy="0.001"
+        iyz="0.0"
+        izz="0.001" />
+        </inertial>
+    </link>
+<!-- Laser 1 Frame -->
+  <link name="lidar1_link">
+    <visual>
+        <origin xyz="0 0 0.031" rpy="0 0 0"/>
+        <geometry>
+            <mesh filename="package://kubot_description/meshes/lidar_frame/$(arg lidar)/laser_link.stl" scale="0.001 0.001 0.001"/>
+        </geometry>
+      <xacro:material_dark_grey/>
+    </visual>
+    <collision>
+        <origin xyz="0 0 0.031" rpy="0 0 0"/>
+        <geometry>
+            <cylinder length="0.0515" radius="0.055"/>
+        </geometry>
+        <xacro:material_white/>
+    </collision>
+    <inertial>
+      <origin xyz="0 0 -0.0241" rpy="0 0 3.1415"/>
+      <mass value="0.179"/>
+      <inertia
+        ixx="0.001"
+        ixy="0.0"
+        ixz="0.0"
+        iyy="0.001"
+        iyz="0.0"
+        izz="0.001" />
+        </inertial>
+    </link>
+<!-- Laser 2 Frame -->
+  <link name="lidar2_link">
+    <visual>
+        <origin xyz="0 0 0.031" rpy="0 0 0"/>
+        <geometry>
+            <mesh filename="package://kubot_description/meshes/lidar_frame/$(arg lidar)/laser_link.stl" scale="0.001 0.001 0.001"/>
+        </geometry>
+      <xacro:material_dark_grey/>
+    </visual>
+    <collision>
+        <origin xyz="0 0 0.031" rpy="0 0 0"/>
+        <geometry>
+            <cylinder length="0.0515" radius="0.055"/>
+        </geometry>
+        <xacro:material_white/>
+    </collision>
+    <inertial>
+      <origin xyz="0 0 -0.0241" rpy="0 0 3.1415"/>
+      <mass value="0.179"/>
+      <inertia
+        ixx="0.001"
+        ixy="0.0"
+        ixz="0.0"
+        iyy="0.001"
+        iyz="0.0"
+        izz="0.001" />
+        </inertial>
+    </link>
+<!-- Define Joint -->
+  <joint name="lidar_joint" type="fixed">
+    <origin xyz="${lidar_joint_xyz}" rpy="${lidar_joint_rpy}" />
+    <parent link="base_link" />
+    <child link="${frame}" />
+  </joint>
+  <joint name="lidar1_joint" type="fixed">
+    <origin xyz="0.319 0.208 0.166" rpy="0 0 0.7854" />
+    <parent link="base_link" />
+    <child link="lidar1_link" />
+  </joint>
+  <joint name="lidar2_joint" type="fixed">
+    <origin xyz="-0.319 -0.208 0.166" rpy="0 0 -2.355" />
+    <parent link="base_link" />
+    <child link="lidar2_link" />
+  </joint>
+<!-- Define Gazebo -->
+  <gazebo reference="${frame}">
+    <material>Gazebo/DarkGrey</material>
+    <sensor type="ray" name="rplidar_a2_ira_sensor">
+    <pose>0 0 0 0 0 0</pose>
+    <visualize>1</visualize>
+    <update_rate>5.5</update_rate>
+    <ray>
+      <scan>
+        <horizontal>
+          <samples>360</samples>
+          <resolution>1</resolution>
+          <min_angle>0.0</min_angle>
+          <max_angle>6.28319</max_angle>
+        </horizontal>
+      </scan>
+      <range>
+        <min>0.15</min>
+        <max>10</max>
+        <resolution>0.01</resolution>
+      </range>
+      <noise>
+        <type>gaussian</type>
+        <mean>0.0</mean>
+        <stddev>0.004</stddev>
+      </noise>
+     </ray>
+     <plugin name="gazebo_ros_rplidar_controller" filename="libgazebo_ros_laser.so">
+        <topicName>scan</topicName>
+        <frameName>${frame}</frameName>
+     </plugin>
+     </sensor>
+  </gazebo>
+  <gazebo reference="lidar1_link">
+    <material>Gazebo/DarkGrey</material>
+    <sensor type="ray" name="lidar1_sensor">
+    <pose>0 0 0 0 0 0</pose>
+    <visualize>1</visualize>
+    <update_rate>5.5</update_rate>
+    <ray>
+      <scan>
+        <horizontal>
+          <samples>360</samples>
+          <resolution>1</resolution>
+          <min_angle>0.0</min_angle>
+          <max_angle>6.28319</max_angle>
+        </horizontal>
+      </scan>
+      <range>
+        <min>0.15</min>
+        <max>10</max>
+        <resolution>0.01</resolution>
+      </range>
+      <noise>
+        <type>gaussian</type>
+        <mean>0.0</mean>
+        <stddev>0.004</stddev>
+      </noise>
+     </ray>
+     <plugin name="gazebo_ros_rplidar_controller" filename="libgazebo_ros_laser.so">
+        <topicName>/lidar1/scan</topicName>
+        <frameName>lidar1_link</frameName>
+     </plugin>
+     </sensor>
+  </gazebo>
+  <gazebo reference="lidar2_link">
+    <material>Gazebo/DarkGrey</material>
+    <sensor type="ray" name="lidar2_sensor">
+    <pose>0 0 0 0 0 0</pose>
+    <visualize>1</visualize>
+    <update_rate>5.5</update_rate>
+    <ray>
+      <scan>
+        <horizontal>
+          <samples>360</samples>
+          <resolution>1</resolution>
+          <min_angle>0.0</min_angle>
+          <max_angle>6.28319</max_angle>
+        </horizontal>
+      </scan>
+      <range>
+        <min>0.15</min>
+        <max>10</max>
+        <resolution>0.01</resolution>
+      </range>
+      <noise>
+        <type>gaussian</type>
+        <mean>0.0</mean>
+        <stddev>0.004</stddev>
+      </noise>
+     </ray>
+     <plugin name="gazebo_ros_rplidar_controller" filename="libgazebo_ros_laser.so">
+        <topicName>/lidar2/scan</topicName>
+        <frameName>lidar2_link</frameName>
+     </plugin>
+     </sensor>
+  </gazebo>
   </xacro:macro>
 </robot>
