Commit message: add view gazebo rviz

File: kubot_description/urdf/model_xacro/kubot2.urdf.xacro (robot description, xacro)
@@ -58,5 +58,5 @@
             <origin xyz="0 0 0" rpy="0 0 0" />
             <geometry>
-                <mesh filename="package://kubot_description/meshes/robot_frame/$(arg model)/logo_frame.stl" scale="0.001 0.001 0.001"/>
+                <box size="0 0 0"/>
             </geometry>
             <xacro:material_white/>

Commit message: debug lidar scan unstable

File: kubot_description/urdf/model_xacro/kubot2.urdf.xacro (robot description, xacro)
@@ -5,11 +5,11 @@
 <xacro:property name="base_radius"  value="0.320"/>
 <xacro:property name="base_length"  value="0.320"/>
-<xacro:property name="base_width"   value="0.140"/>
+<xacro:property name="base_width"   value="0.145"/>
 <xacro:property name="wheel_mass"    value="0.05"/>
-<xacro:property name="wheel_radius"  value="0.081"/>
+<xacro:property name="wheel_radius"  value="0.0815"/>
 <xacro:property name="wheel_length"  value="0.020"/>
 <xacro:property name="wheel_joint_x" value="0.00"/>
 <xacro:property name="wheel_joint_y" value="0.122"/>
-<xacro:property name="wheel_joint_z" value="0.08"/>
+<xacro:property name="wheel_joint_z" value="0.080"/>
 <xacro:property name="caster_mass"    value="0.01"/>
 <xacro:property name="caster_radius"  value="0.015"/>
@@ -31,5 +31,5 @@
             <origin xyz="-0.05 0 ${base_width/2+0.02}" rpy="0 0 0" />
             <geometry>
-                <box size="${base_radius} ${base_length} ${base_width}"/>
+               <cylinder length="${base_width}" radius="${base_radius/1.6}"/>
             </geometry>
         </collision>
@@ -46,10 +46,27 @@
         </inertial>
     </link>
+<!-- R1 Frame a.k.a adornment -->
+    <link name= "r1_frame">
+        <visual>
+            <origin xyz="0 0 0" rpy="0 0 0" />
+            <geometry>
+                <mesh filename="package://kubot_description/meshes/robot_frame/$(arg model)/r1_frame.stl" scale="0.001 0.001 0.001"/>
+            </geometry>
+            <xacro:material_orange/>
+        </visual>
+        <collision>
+            <origin xyz="0 0 0" rpy="0 0 0" />
+            <geometry>
+                <box size="0.0001 0.0001 0.0001"/>
+            </geometry>
+        </collision>
+        <xacro:box_inertial_matrix m="0" a="0" b="0" c="0"/>
+    </link>
 <!-- Logo Frame a.k.a adornment -->
     <link name= "logo_frame">
         <visual>
-            <origin xyz="0 0 0" rpy="0 0 0" />
-            <geometry>
-                <mesh filename="package://kubot_description/meshes/robot_frame/$(arg model)/logo_frame.stl" scale="0.001 0.001 0.001"/>
+            <origin xyz="0.01 0 0" rpy="0 0 0" />
+            <geometry>
+                <mesh filename="package://kubot_description/meshes/robot_frame/$(arg model)/logo_frame.stl" scale="0.0015 0.0015 0.001"/>
             </geometry>
             <xacro:material_white/>
@@ -58,7 +75,6 @@
             <origin xyz="0 0 0" rpy="0 0 0" />
             <geometry>
-                <mesh filename="package://kubot_description/meshes/robot_frame/$(arg model)/logo_frame.stl" scale="0.001 0.001 0.001"/>
-            </geometry>
-            <xacro:material_white/>
+                <box size="0.0001 0.0001 0.0001"/>
+            </geometry>
         </collision>
         <xacro:box_inertial_matrix m="0" a="0" b="0" c="0"/>
@@ -78,5 +94,4 @@
                     <cylinder length="${wheel_length}" radius="${wheel_radius}"/>
               </geometry>
-              <xacro:material_white/>
         </collision>
         <xacro:cylinder_inertial_matrix m="${wheel_mass}" r="${wheel_radius}" h="${wheel_length}"/>
@@ -96,5 +111,4 @@
                     <cylinder length="${wheel_length}" radius="${wheel_radius}"/>
               </geometry>
-              <xacro:material_white/>
         </collision>
         <xacro:cylinder_inertial_matrix m="${wheel_mass}" r="${wheel_radius}" h="${wheel_length}"/>
@@ -118,4 +132,8 @@
     </link>
 <!-- Define Joint -->
+    <joint name="r1_joint" type="fixed">
+        <parent link="base_link"/>
+        <child link="r1_frame"/>
+    </joint>
     <joint name="logo_joint" type="fixed">
         <parent link="base_link"/>
@@ -141,4 +159,7 @@
 <!-- Define Gazebo -->
     <gazebo reference="base_link">
+        <material>Gazebo/Orange</material>
+    </gazebo>
+    <gazebo reference="r1_frame">
         <material>Gazebo/Orange</material>
     </gazebo>
@@ -162,5 +183,5 @@
         <kd>1.0</kd>
         <minDepth>0.001</minDepth>
-        <maxVel>0.01</maxVel>
+        <maxVel>1.0</maxVel>
         <fdir1>0 1 0</fdir1>
         <material>Gazebo/Black</material>

File: kubot_description/urdf/model_xacro/neuronbot2.urdf.xacro (robot description, xacro)
@@ -7,5 +7,5 @@
 <xacro:property name="base_width"   value="0.200"/>
 <xacro:property name="wheel_mass"    value="0.05"/>
-<xacro:property name="wheel_radius"  value="0.0425"/>
+<xacro:property name="wheel_radius"  value="0.042"/>
 <xacro:property name="wheel_length"  value="0.02"/>
 <xacro:property name="wheel_joint_x" value="0"/>
@@ -58,7 +58,6 @@
             <origin xyz="0 0 0" rpy="0 0 0" />
             <geometry>
-                <mesh filename="package://kubot_description/meshes/robot_frame/$(arg model)/r1_frame.stl" scale="0.001 0.001 0.001"/>
-            </geometry>
-            <xacro:material_white/>
+                <box size="0.0001 0.0001 0.0001"/>
+            </geometry>
         </collision>
         <xacro:box_inertial_matrix m="0" a="0" b="0" c="0"/>
@@ -76,7 +75,6 @@
             <origin xyz="0 0 0" rpy="0 0 0" />
             <geometry>
-                <mesh filename="package://kubot_description/meshes/robot_frame/$(arg model)/logo_frame.stl" scale="0.001 0.001 0.001"/>
-            </geometry>
-            <xacro:material_white/>
+                <box size="0.0001 0.0001 0.0001"/>
+            </geometry>
         </collision>
         <xacro:box_inertial_matrix m="0" a="0" b="0" c="0"/>
@@ -92,9 +90,8 @@
         </visual>
         <collision>
-              <origin xyz="0 ${-1*wheel_length/2} 0" rpy="${M_PI/2} 0 0"/>
-              <geometry>
-                    <cylinder length="${wheel_length}" radius="${wheel_radius}"/>
-              </geometry>
-              <xacro:material_white/>
+            <origin xyz="0 ${-1*wheel_length/2} 0" rpy="${M_PI/2} 0 0"/>
+            <geometry>
+                <cylinder length="${wheel_length}" radius="${wheel_radius}"/>
+            </geometry>
         </collision>
         <xacro:cylinder_inertial_matrix m="${wheel_mass}" r="${wheel_radius}" h="${wheel_length}"/>
@@ -110,9 +107,9 @@
         </visual>
         <collision>
-              <origin xyz="0 ${-1*wheel_length/2} 0" rpy="${M_PI/2} 0 0"/>
-              <geometry>
-                    <cylinder length="${wheel_length}" radius="${wheel_radius}"/>
-              </geometry>
-              <xacro:material_white/>
+            <origin xyz="0 ${-1*wheel_length/2} 0" rpy="${M_PI/2} 0 0"/>
+            <geometry>
+                <cylinder length="${wheel_length}" radius="${wheel_radius}"/>
+            </geometry>
+            <xacro:material_white/>
         </collision>
         <xacro:cylinder_inertial_matrix m="${wheel_mass}" r="${wheel_radius}" h="${wheel_length}"/>
@@ -209,5 +206,5 @@
         <kd>1.0</kd>
         <minDepth>0.001</minDepth>
-        <maxVel>0.01</maxVel>
+        <maxVel>1.0</maxVel>
         <fdir1>0 1 0</fdir1>
         <material>Gazebo/Red</material>

Commit message: test

File: kubot_description/urdf/model_xacro/kubot2.urdf.xacro (robot description, xacro)
@@ -9,4 +9,5 @@
 <xacro:property name="wheel_radius"  value="0.0815"/>
 <xacro:property name="wheel_length"  value="0.020"/>
+<xacro:property name="wheel_width"   value="0.0"/>
 <xacro:property name="wheel_joint_x" value="0.00"/>
 <xacro:property name="wheel_joint_y" value="0.122"/>
@@ -15,4 +16,5 @@
 <xacro:property name="caster_radius"  value="0.015"/>
 <xacro:property name="caster_length"  value="0.02"/>
+<xacro:property name="caster_width"   value="0.3"/>
 <xacro:property name="caster_joint_x" value="0.164"/>
 <xacro:property name="caster_joint_y" value="0.0"/>
@@ -90,8 +92,8 @@
         </visual>
         <collision>
-              <origin xyz="0 0 0" rpy="${M_PI/2} 0 0"/>
-              <geometry>
-                    <cylinder length="${wheel_length}" radius="${wheel_radius}"/>
-              </geometry>
+            <origin xyz="0 0 0" rpy="${M_PI/2} 0 0"/>
+            <geometry>
+                <cylinder length="${wheel_length}" radius="${wheel_radius}"/>
+            </geometry>
         </collision>
         <xacro:cylinder_inertial_matrix m="${wheel_mass}" r="${wheel_radius}" h="${wheel_length}"/>
@@ -107,8 +109,8 @@
         </visual>
         <collision>
-              <origin xyz="0 0 0" rpy="${M_PI/2} 0 0"/>
-              <geometry>
-                    <cylinder length="${wheel_length}" radius="${wheel_radius}"/>
-              </geometry>
+            <origin xyz="0 0 0" rpy="${M_PI/2} 0 0"/>
+            <geometry>
+                <cylinder length="${wheel_length}" radius="${wheel_radius}"/>
+            </geometry>
         </collision>
         <xacro:cylinder_inertial_matrix m="${wheel_mass}" r="${wheel_radius}" h="${wheel_length}"/>
