Commit message: update galitay2

File: kubot_description/urdf/model_xacro/galiray2.urdf.xacro (robot description, xacro)
@@ -4,9 +4,9 @@
 	<xacro:include filename="$(find kubot_description)/urdf/kubot_properties.urdf.xacro" />
 	<xacro:property name="base_mass" value="4.2" />
-	<xacro:property name="base_radius" value="0.39" />
+	<xacro:property name="base_radius" value="0.33" />
 	<xacro:property name="base_length" value="0.33" />
 	<xacro:property name="base_width" value="0.2" />
 	<xacro:property name="wheel_mass" value="0.1" />
-	<xacro:property name="wheel_radius" value="0.033" />
+	<xacro:property name="wheel_radius" value="0.05" />
 	<xacro:property name="wheel_length" value="0.04" />
 	<xacro:property name="wheel_width" value="0.0" />
