Commit message: udpate

File: kubot_description/urdf/model_xacro/aider.urdf.xacro (robot description, xacro)
@@ -321,15 +321,9 @@
     </gazebo>
   </xacro:macro>
-  <!-- Lidar Frame a.k.a Lidar Pos-->
-  <xacro:property name="lidar_joint_xyz" value="0 0 0.166"/>
-  <xacro:property name="lidar_joint_rpy" value="0 0 0"/>
-  <!-- Camera a.k.a Camera Pos -->
-  <xacro:property name="camera_pos_rear" value="false"/>
-  <xacro:if value="${camera_pos_rear}">
-    <xacro:property name="camera_joint_xyz" value="0.26 0 0.17"/>
-  </xacro:if>
-  <xacro:unless value="${camera_pos_rear}">
-    <xacro:property name="camera_joint_xyz" value="0 0 0"/>
-  </xacro:unless>
-  <xacro:property name="camera_joint_rpy" value="0 0 0"/>
+<!-- Lidar Frame a.k.a Lidar Pos-->
+<xacro:property name="lidar_joint_xyz" value="0 0 0.227"/>
+<xacro:property name="lidar_joint_rpy" value="0 0 0"/>
+<!-- Camera a.k.a Camera Pos -->
+<xacro:property name="camera_joint_xyz" value="0.26 0 0.17"/>
+<xacro:property name="camera_joint_rpy" value="0 0 0"/>
 </robot>

File: kubot_description/urdf/model_xacro/kubot2.urdf.xacro (robot description, xacro)
@@ -175,7 +175,7 @@
     </gazebo>
 </xacro:macro>
-  <!-- Lidar Frame a.k.a Lidar Pos-->
-  <xacro:property name="lidar_joint_xyz" value="-0.05 0 0.194"/>
-  <xacro:property name="lidar_joint_rpy" value="0 0 0"/>
+<!-- Lidar Frame a.k.a Lidar Pos-->
+<xacro:property name="lidar_joint_xyz" value="-0.05 0 0.194"/>
+<xacro:property name="lidar_joint_rpy" value="0 0 0"/>
 <!-- Camera a.k.a Camera Pos -->
 <xacro:property name="camera_joint_xyz" value="0.1 0 0.14"/>

Commit message: update

File: kubot_description/urdf/model_xacro/aider.urdf.xacro (robot description, xacro)
@@ -2,5 +2,5 @@
 <robot name="kubot_robot" xmlns:xacro="https://ros.org/wiki/xacro">
 <xacro:include filename="$(find kubot_description)/urdf/kubot_properties.urdf.xacro"/>
-<xacro:property name="base_mass"    value="100"/>
+<xacro:property name="base_mass"    value="80"/>
 <xacro:property name="base_radius"  value="0.793"/>
 <xacro:property name="base_length"  value="0.530"/>
@@ -12,5 +12,5 @@
 <xacro:property name="wheel_joint_y" value="0.220"/>
 <xacro:property name="wheel_joint_z" value="0.075"/>
-<xacro:property name="caster_mass"    value="2"/>
+<xacro:property name="caster_mass"    value="0.01"/>
 <xacro:property name="caster_radius"  value="0.0385"/>
 <xacro:property name="caster_length"  value="0.05"/>
@@ -45,5 +45,5 @@
             izz="${base_mass*(base_radius*base_radius+base_length*base_length)/12}" />
         </inertial>
-        </link>
+    </link>
 <!-- R1 Frame a.k.a adornment -->
     <link name= "r1_frame">
@@ -253,5 +253,5 @@
         <kd>1.0</kd>
         <minDepth>0.001</minDepth>
-        <maxVel>0.01</maxVel>
+        <maxVel>1.0</maxVel>
         <fdir1>0 1 0</fdir1>
         <material>Gazebo/Black</material>
@@ -316,5 +316,5 @@
             <wheelDiameter>${2*wheel_radius}</wheelDiameter>
             <wheelAcceleration>1</wheelAcceleration>
-            <wheelTorque>10</wheelTorque>
+            <wheelTorque>60</wheelTorque>
             <rosDebugLevel>na</rosDebugLevel>
         </plugin>

File: kubot_description/urdf/model_xacro/wagv.urdf.xacro (robot description, xacro)
@@ -5,10 +5,10 @@
 <xacro:property name="base_radius"  value="0.755"/>
 <xacro:property name="base_length"  value="0.675"/>
-<xacro:property name="base_width"   value="0.190"/>
-<xacro:property name="wheel_mass"    value="2"/>
-<xacro:property name="wheel_radius"  value="0.0770"/>
+<xacro:property name="base_width"   value="0.200"/>
+<xacro:property name="wheel_mass"    value="0.5"/>
+<xacro:property name="wheel_radius"  value="0.0765"/>
 <xacro:property name="wheel_length"  value="0.05"/>
 <xacro:property name="wheel_joint_x" value="0"/>
-<xacro:property name="wheel_joint_y" value="0.275"/>
+<xacro:property name="wheel_joint_y" value="0.280"/>
 <xacro:property name="wheel_joint_z" value="0.075"/>
 <xacro:property name="caster_mass"    value="0.1"/>
@@ -16,5 +16,5 @@
 <xacro:property name="caster_length"  value="0.05"/>
 <xacro:property name="caster_joint_x" value="0.268"/>
-<xacro:property name="caster_joint_y" value="0.185"/>
+<xacro:property name="caster_joint_y" value="0.175"/>
 <xacro:property name="caster_joint_z" value="0.028"/>
 <xacro:macro name="base">
@@ -45,5 +45,5 @@
             izz="${base_mass*(base_radius*base_radius+base_length*base_length)/12}" />
         </inertial>
-        </link>
+    </link>
 <!-- R1 Frame a.k.a adornment -->
     <link name= "r1_frame">
@@ -125,5 +125,5 @@
                 <mesh filename="package://kubot_description/meshes/robot_frame/$(arg model)/wheel_link.stl" scale="0.001 0.001 0.001"/>
             </geometry>
-            <xacro:material_red/>
+            <xacro:material_black/>
         </visual>
         <collision>
@@ -143,5 +143,5 @@
                 <mesh filename="package://kubot_description/meshes/robot_frame/$(arg model)/wheel_link.stl" scale="0.001 0.001 0.001"/>
             </geometry>
-            <xacro:material_red/>
+            <xacro:material_black/>
         </visual>
         <collision>
@@ -303,5 +303,5 @@
         <kd>1.0</kd>
         <minDepth>0.001</minDepth>
-        <maxVel>0.01</maxVel>
+        <maxVel>1.0</maxVel>
         <fdir1>0 1 0</fdir1>
         <material>Gazebo/Black</material>
@@ -366,20 +366,14 @@
             <wheelDiameter>${2*wheel_radius}</wheelDiameter>
             <wheelAcceleration>1</wheelAcceleration>
-            <wheelTorque>10</wheelTorque>
+            <wheelTorque>60</wheelTorque>
             <rosDebugLevel>na</rosDebugLevel>
         </plugin>
     </gazebo>
   </xacro:macro>
-  <!-- Lidar Frame a.k.a Lidar Pos-->
-  <xacro:property name="lidar_joint_xyz" value="0.27 0 0.26"/>
-  <xacro:property name="lidar_joint_rpy" value="0 0 0"/>
-  <!-- Camera a.k.a Camera Pos -->
-  <xacro:property name="camera_pos_rear" value="false"/>
-  <xacro:if value="${camera_pos_rear}">
-    <xacro:property name="camera_joint_xyz" value="0.26 0 0.17"/>
-  </xacro:if>
-  <xacro:unless value="${camera_pos_rear}">
-    <xacro:property name="camera_joint_xyz" value="0 0 0"/>
-  </xacro:unless>
-  <xacro:property name="camera_joint_rpy" value="0 0 0"/>
+<!-- Lidar Frame a.k.a Lidar Pos-->
+<xacro:property name="lidar_joint_xyz" value="0.27 0 0.26"/>
+<xacro:property name="lidar_joint_rpy" value="0 0 0"/>
+<!-- Camera a.k.a Camera Pos -->
+<xacro:property name="camera_joint_xyz" value="0.26 0 0.17"/>
+<xacro:property name="camera_joint_rpy" value="0 0 0"/>
 </robot>

Commit message: update aider robot rviz

File: kubot_description/urdf/model_xacro/aider.urdf.xacro (robot description, xacro)
@@ -26,5 +26,5 @@
                     <mesh filename="package://kubot_description/meshes/robot_frame/$(arg model)/base_link.stl" scale="0.001 0.001 0.001" />
                 </geometry>
-                <xacro:material_light_blue />
+                <xacro:material_white />
             </visual>
             <collision>
@@ -47,5 +47,5 @@
                     <mesh filename="package://kubot_description/meshes/robot_frame/$(arg model)/r1_frame.stl" scale="0.001 0.001 0.001" />
                 </geometry>
-                <xacro:material_white />
+                <xacro:material_dark_blue />
             </visual>
             <collision>
@@ -54,5 +54,4 @@
                     <mesh filename="package://kubot_description/meshes/robot_frame/$(arg model)/r1_frame.stl" scale="0.001 0.001 0.001" />
                 </geometry>
-                <xacro:material_white />
             </collision>
             <xacro:box_inertial_matrix m="0" a="0" b="0" c="0" />
@@ -65,5 +64,5 @@
                     <mesh filename="package://kubot_description/meshes/robot_frame/$(arg model)/r2_frame.stl" scale="0.001 0.001 0.001" />
                 </geometry>
-                <xacro:material_dark_blue />
+                <xacro:material_black />
             </visual>
             <collision>
@@ -72,5 +71,21 @@
                     <mesh filename="package://kubot_description/meshes/robot_frame/$(arg model)/r2_frame.stl" scale="0.001 0.001 0.001" />
                 </geometry>
-                <xacro:material_white />
+            </collision>
+            <xacro:box_inertial_matrix m="0" a="0" b="0" c="0" />
+        </link>
+        <!-- R3 Frame a.k.a adornment -->
+        <link name="r3_frame">
+            <visual>
+                <origin xyz="0 0 0" rpy="0 0 0" />
+                <geometry>
+                    <mesh filename="package://kubot_description/meshes/robot_frame/$(arg model)/r3_frame.stl" scale="0.001 0.001 0.001" />
+                </geometry>
+                <xacro:material_yellow />
+            </visual>
+            <collision>
+                <origin xyz="0 0 0" rpy="0 0 0" />
+                <geometry>
+                    <mesh filename="package://kubot_description/meshes/robot_frame/$(arg model)/r3_frame.stl" scale="0.001 0.001 0.001" />
+                </geometry>
             </collision>
             <xacro:box_inertial_matrix m="0" a="0" b="0" c="0" />
@@ -119,5 +134,5 @@
                     <sphere radius="${caster_radius}" />
                 </geometry>
-                <xacro:material_white />
+                <xacro:material_red />
             </visual>
             <collision>
@@ -136,5 +151,5 @@
                     <sphere radius="${caster_radius}" />
                 </geometry>
-                <xacro:material_white />
+                <xacro:material_red />
             </visual>
             <collision>
@@ -153,5 +168,5 @@
                     <sphere radius="${caster_radius}" />
                 </geometry>
-                <xacro:material_white />
+                <xacro:material_red />
             </visual>
             <collision>
@@ -170,5 +185,5 @@
                     <sphere radius="${caster_radius}" />
                 </geometry>
-                <xacro:material_white />
+                <xacro:material_red />
             </visual>
             <collision>
@@ -188,4 +203,8 @@
             <parent link="base_link" />
             <child link="r2_frame" />
+        </joint>
+        <joint name="r3_joint" type="fixed">
+            <parent link="base_link" />
+            <child link="r3_frame" />
         </joint>
         <joint name="wheel_right_joint" type="continuous">
@@ -223,11 +242,14 @@
         <!-- Define Gazebo -->
         <gazebo reference="base_link">
-            <material>Gazebo/SkyBlue</material>
+            <material>Gazebo/White</material>
         </gazebo>
         <gazebo reference="r1_frame">
-            <material>Gazebo/White</material>
+            <material>Gazebo/Blue</material>
         </gazebo>
         <gazebo reference="r2_frame">
-            <material>Gazebo/Blue</material>
+            <material>Gazebo/Black</material>
+        </gazebo>
+        <gazebo reference="r3_frame">
+            <material>Gazebo/Yellow</material>
         </gazebo>
         <gazebo reference="wheel_right_link">

Commit message: update collision

File: kubot_description/urdf/model_xacro/aider.urdf.xacro (robot description, xacro)
@@ -49,4 +49,10 @@
                 <xacro:material_dark_blue />
             </visual>
+            <collision>
+                <origin xyz="0 0 0.18" rpy="0 0 0" />
+                <geometry>
+                    <box size="0.65 0.405 0.092" />
+                </geometry>
+            </collision>
         </link>
         <!-- R2 Frame a.k.a adornment -->

Commit message: update aider camera

File: kubot_description/urdf/model_xacro/aider.urdf.xacro (robot description, xacro)
@@ -332,5 +332,5 @@
     <xacro:property name="lidar_joint_rpy" value="0 0 0" />
     <!-- Camera a.k.a Camera Pos -->
-    <xacro:property name="camera_joint_xyz" value="0.38 0 0.08" />
-    <xacro:property name="camera_joint_rpy" value="0 0 0" />
+    <xacro:property name="camera_joint_xyz" value="-0.39 0 0.235" />
+    <xacro:property name="camera_joint_rpy" value="0 0 3.14" />
 </robot>
