Commit message: update fullon robot mind aix

File: kubot_description/urdf/model_xacro/fullon.urdf.xacro (robot description, xacro)
@@ -11,5 +11,5 @@
 	<xacro:property name="wheel_length" value="0.050" />
 	<xacro:property name="wheel_width" value="0.0" />
-	<xacro:property name="wheel_joint_x" value="0.080" />
+	<xacro:property name="wheel_joint_x" value="0.0" />
 	<xacro:property name="wheel_joint_y" value="0.245" />
 	<xacro:property name="wheel_joint_z" value="0.075" />
@@ -18,5 +18,5 @@
 	<xacro:property name="caster_length" value="0.02" />
 	<xacro:property name="caster_width" value="0.05" />
-	<xacro:property name="caster_joint_x" value="0.170" />
+	<xacro:property name="caster_joint_x" value="0.25" />
 	<xacro:property name="caster_joint_y" value="0.0" />
 	<xacro:property name="caster_joint_z" value="0.025" />
@@ -25,5 +25,5 @@
 		<link name="base_link">
 			<visual>
-				<origin xyz="0 0 ${base_length/2+0.04}" rpy="0 0 0" />
+				<origin xyz="-0.08 0 ${base_length/2+0.04}" rpy="0 0 0" />
 				<geometry>
 					<cylinder length="${base_length}" radius="${base_radius}" />
@@ -32,5 +32,5 @@
 			</visual>
 			<collision>
-				<origin xyz="0 0 ${base_length/2+0.04}" rpy="0 0 0" />
+				<origin xyz="-0.08 0 ${base_length/2+0.04}" rpy="0 0 0" />
 				<geometry>
 					<cylinder length="${base_length}" radius="${base_radius}" />
@@ -38,5 +38,5 @@
 			</collision>
 			<inertial>
-				<origin xyz="0 0 ${base_length/2+0.04}" rpy="0 0 0" />
+				<origin xyz="-0.08 0 ${base_length/2+0.04}" rpy="0 0 0" />
 				<xacro:cylinder_inertial_matrix m="${base_mass}" r="${base_radius}" h="${base_length}" />
 			</inertial>
@@ -184,5 +184,5 @@
 	</xacro:macro>
 	<!-- Lidar Frame a.k.a Lidar Pos-->
-	<xacro:property name="lidar_joint_xyz" value="0.19 0 0.42" />
+	<xacro:property name="lidar_joint_xyz" value="0.11 0 0.42" />
 	<xacro:property name="lidar_joint_rpy" value="0 0 0" />
 	<!-- Camera a.k.a Camera Pos -->

Commit message: update wheel dis

File: kubot_description/urdf/model_xacro/fullon.urdf.xacro (robot description, xacro)
@@ -12,5 +12,5 @@
 	<xacro:property name="wheel_width" value="0.0" />
 	<xacro:property name="wheel_joint_x" value="0.0" />
-	<xacro:property name="wheel_joint_y" value="0.245" />
+	<xacro:property name="wheel_joint_y" value="0.240" />
 	<xacro:property name="wheel_joint_z" value="0.075" />
 	<xacro:property name="caster_mass" value="0.05" />
@@ -184,5 +184,5 @@
 	</xacro:macro>
 	<!-- Lidar Frame a.k.a Lidar Pos-->
-	<xacro:property name="lidar_joint_xyz" value="0.11 0 0.42" />
+	<xacro:property name="lidar_joint_xyz" value="0.12 0 0.42" />
 	<xacro:property name="lidar_joint_rpy" value="0 0 0" />
 	<!-- Camera a.k.a Camera Pos -->
