Commit message: ?

File: kubot_description/urdf/lidar_xacro/rplidar-a1.urdf.xacro (robot description, xacro)
@@ -39,5 +39,5 @@
     <child link="${frame}" />
   </joint>
-<!-- Define Gazebo -->
+<!-- Define Gazebo (ｏ´・ε・｀ｏ) -->
   <gazebo reference="${frame}">
     <material>Gazebo/DarkGrey</material>
@@ -51,6 +51,6 @@
           <samples>360</samples>
           <resolution>1</resolution>
-          <min_angle>0.0</min_angle>
-          <max_angle>6.28319</max_angle>
+          <min_angle>-3.14159</min_angle>
+          <max_angle>3.14159</max_angle>
         </horizontal>
       </scan>
@@ -58,10 +58,10 @@
         <min>0.15</min>
         <max>10</max>
-        <resolution>0.01</resolution>
+        <resolution>0.05</resolution>
       </range>
       <noise>
         <type>gaussian</type>
         <mean>0.0</mean>
-        <stddev>0.004</stddev>
+        <stddev>0.01</stddev>
       </noise>
      </ray>

File: kubot_description/urdf/model_xacro/kubot2.urdf.xacro (robot description, xacro)
@@ -58,5 +58,5 @@
             <origin xyz="0 0 0" rpy="0 0 0" />
             <geometry>
-                <box size="0 0 0"/>
+                <mesh filename="package://kubot_description/meshes/robot_frame/$(arg model)/logo_frame.stl" scale="0.001 0.001 0.001"/>
             </geometry>
             <xacro:material_white/>

Commit message: update

File: kubot_description/urdf/lidar_xacro/rplidar-a1.urdf.xacro (robot description, xacro)
@@ -57,5 +57,5 @@
       <range>
         <min>0.15</min>
-        <max>10</max>
+        <max>12</max>
         <resolution>0.05</resolution>
       </range>
@@ -63,8 +63,8 @@
         <type>gaussian</type>
         <mean>0.0</mean>
-        <stddev>0.01</stddev>
+        <stddev>0.004</stddev>
       </noise>
      </ray>
-     <plugin name="gazebo_ros_rplidar_controller" filename="libgazebo_ros_laser.so">
+     <plugin name="gazebo_ros_rplidar_a1_controller" filename="libgazebo_ros_laser.so">
         <topicName>scan</topicName>
         <frameName>${frame}</frameName>

File: kubot_description/urdf/lidar_xacro/rplidar-a2.urdf.xacro (robot description, xacro)
@@ -1,44 +1,75 @@
 <?xml version="1.0"?>
-<robot name="kubot" xmlns:xacro="https://ros.org/wiki/xacro">
-  <xacro:include filename="$(find kubot_description)/urdf/kubot_properties.urdf.xacro"/>
-  <xacro:macro
-  name="lidar"
-  params="frame:=laser_link lidar_enabled:=true lidar_joint_xyz:=0 lidar_joint_rpy:=0">
-      <xacro:if value="${lidar_enabled}">
-        <!-- laser link -->
-        <link name="${frame}">
-            <visual>
-                <origin xyz="0 0 0.031" rpy="0 0 0"/>
-                <geometry>
-                    <mesh filename="package://kubot_description/meshes/lidar_frame/rplidar-a2/laser_link.stl" scale="0.001 0.001 0.001"/>
-                </geometry>
-            <xacro:material_dark_grey/>
-            </visual>
-            <collision>
-                <origin xyz="0 0 0.031" rpy="0 0 0"/>
-                <geometry>
-                    <mesh filename="package://kubot_description/meshes/lidar_frame/rplidar-a2/laser_link.stl" scale="0.001 0.001 0.001"/>
-                </geometry>
-            <xacro:material_white/>
-            </collision>
-            <inertial>
-                <origin xyz="0 0 0.031" rpy="0 0 0"/>
-                <mass value="0.179"/>
-                <inertia
-                   ixx="0.00028"
-                   ixy="0.0"
-                   ixz="0.0"
-                   iyy="0.00028"
-                   iyz="0.0"
-                   izz="0.00022" />
-            </inertial>
-        </link>
-        <!-- lidar joint -->
-        <joint name="lidar_joint" type="fixed">
-            <origin xyz="${lidar_joint_xyz}" rpy="${lidar_joint_rpy}" />
-            <parent link="base_link" />
-            <child link="${frame}" />
-        </joint>
-      </xacro:if>
-  </xacro:macro>
+<robot name="kubot_robot" xmlns:xacro="https://ros.org/wiki/xacro">
+<xacro:include filename="$(find kubot_description)/urdf/kubot_properties.urdf.xacro"/>
+<xacro:macro
+name="lidar"
+params="frame:=laser_link lidar_joint_xyz:=0 lidar_joint_rpy:=0">
+<!-- Laser Frame -->
+  <link name="${frame}">
+    <visual>
+        <origin xyz="0 0 0" rpy="0 0 0"/>
+        <geometry>
+            <mesh filename="package://kubot_description/meshes/lidar_frame/$(arg lidar)/laser_link.stl" scale="0.001 0.001 0.001"/>
+        </geometry>
+      <xacro:material_dark_grey/>
+    </visual>
+    <collision>
+        <origin xyz="0 0 0" rpy="0 0 0"/>
+        <geometry>
+            <cylinder length="0.0415" radius="0.035"/>
+        </geometry>
+        <xacro:material_white/>
+    </collision>
+    <inertial>
+      <origin xyz="0 0 0" rpy="0 0 3.1415"/>
+      <mass value="0.179"/>
+      <inertia
+        ixx="0.001"
+        ixy="0.0"
+        ixz="0.0"
+        iyy="0.001"
+        iyz="0.0"
+        izz="0.001" />
+        </inertial>
+    </link>
+<!-- Define Joint -->
+    <joint name="lidar_joint" type="fixed">
+        <origin xyz="${lidar_joint_xyz}" rpy="${lidar_joint_rpy}" />
+        <parent link="base_link" />
+        <child link="${frame}" />
+    </joint>
+<!-- Define Gazebo -->
+    <gazebo reference="${frame}">
+        <material>Gazebo/DarkGrey</material>
+        <sensor type="ray" name="rplidar_a2_sensor">
+        <pose>0 0 0 0 0 0</pose>
+        <visualize>1</visualize>
+        <update_rate>10</update_rate>
+        <ray>
+            <scan>
+                <horizontal>
+                    <samples>360</samples>
+                    <resolution>1</resolution>
+                    <min_angle>0.0</min_angle>
+                    <max_angle>6.28319</max_angle>
+                </horizontal>
+            </scan>
+            <range>
+                <min>0.15</min>
+                <max>12</max>
+                <resolution>0.01</resolution>
+            </range>
+            <noise>
+                <type>gaussian</type>
+                <mean>0.0</mean>
+                <stddev>0.004</stddev>
+            </noise>
+        </ray>
+        <plugin name="gazebo_ros_rplidar_a2_controller" filename="libgazebo_ros_laser.so">
+            <topicName>scan</topicName>
+            <frameName>${frame}</frameName>
+        </plugin>
+        </sensor>
+    </gazebo>
+</xacro:macro>
 </robot>

File: kubot_description/urdf/lidar_xacro/sick-tim551.urdf.xacro (robot description, xacro)
@@ -45,5 +45,5 @@
     <pose>0 0 0 0 0 0</pose>
     <visualize>1</visualize>
-    <update_rate>10</update_rate>
+    <update_rate>30</update_rate>
     <ray>
       <scan>
@@ -66,5 +66,5 @@
       </noise>
      </ray>
-     <plugin name="gazebo_ros_rplidar_controller" filename="libgazebo_ros_laser.so">
+     <plugin name="gazebo_ros_sick_tim551_controller" filename="libgazebo_ros_laser.so">
         <topicName>scan</topicName>
         <frameName>${frame}</frameName>

File: kubot_description/urdf/lidar_xacro/two-rplidar-a2.urdf.xacro (robot description, xacro)
@@ -111,5 +111,5 @@
     <pose>0 0 0 0 0 0</pose>
     <visualize>1</visualize>
-    <update_rate>5.5</update_rate>
+    <update_rate>10</update_rate>
     <ray>
       <scan>
@@ -122,6 +122,6 @@
       </scan>
       <range>
-        <min>0.12</min>
-        <max>10</max>
+        <min>0.15</min>
+        <max>12</max>
         <resolution>0.01</resolution>
       </range>
@@ -132,5 +132,5 @@
       </noise>
      </ray>
-     <plugin name="gazebo_ros_rplidar_controller" filename="libgazebo_ros_laser.so">
+     <plugin name="gazebo_ros_rplidar_controller1" filename="libgazebo_ros_laser.so">
         <topicName>/lidar1/scan</topicName>
         <frameName>lidar1_link</frameName>
@@ -143,5 +143,5 @@
     <pose>0 0 0 0 0 0</pose>
     <visualize>1</visualize>
-    <update_rate>5.5</update_rate>
+    <update_rate>10</update_rate>
     <ray>
       <scan>
@@ -154,7 +154,7 @@
       </scan>
       <range>
-        <min>0.12</min>
-        <max>10</max>
-        <resolution>0.01</resolution>
+        <min>0.15</min>
+        <max>12</max>
+        <resolution>0.001</resolution>
       </range>
       <noise>
@@ -164,5 +164,5 @@
       </noise>
      </ray>
-     <plugin name="gazebo_ros_rplidar_controller" filename="libgazebo_ros_laser.so">
+     <plugin name="gazebo_ros_rplidar_controller2" filename="libgazebo_ros_laser.so">
         <topicName>/lidar2/scan</topicName>
         <frameName>lidar2_link</frameName>

File: kubot_description/urdf/model_xacro/aider.urdf.xacro (robot description, xacro)
@@ -325,5 +325,5 @@
 <xacro:property name="lidar_joint_rpy" value="0 0 0"/>
 <!-- Camera a.k.a Camera Pos -->
-<xacro:property name="camera_joint_xyz" value="0.26 0 0.17"/>
+<xacro:property name="camera_joint_xyz" value="0.38 0 0.08"/>
 <xacro:property name="camera_joint_rpy" value="0 0 0"/>
 </robot>

File: kubot_description/urdf/model_xacro/kubot2.urdf.xacro (robot description, xacro)
@@ -3,9 +3,9 @@
 <xacro:include filename="$(find kubot_description)/urdf/kubot_properties.urdf.xacro"/>
 <xacro:property name="base_mass"    value="4.2"/>
-<xacro:property name="base_radius"  value="0.300"/>
-<xacro:property name="base_length"  value="0.300"/>
+<xacro:property name="base_radius"  value="0.320"/>
+<xacro:property name="base_length"  value="0.320"/>
 <xacro:property name="base_width"   value="0.140"/>
 <xacro:property name="wheel_mass"    value="0.05"/>
-<xacro:property name="wheel_radius"  value="0.080"/>
+<xacro:property name="wheel_radius"  value="0.081"/>
 <xacro:property name="wheel_length"  value="0.020"/>
 <xacro:property name="wheel_joint_x" value="0.00"/>
@@ -45,5 +45,5 @@
             izz="${base_mass*(base_radius*base_radius+base_length*base_length)/12}" />
         </inertial>
-        </link>
+    </link>
 <!-- Logo Frame a.k.a adornment -->
     <link name= "logo_frame">

Commit message: udpate kubot xacro

File: kubot_description/urdf/lidar_xacro/rplidar-a1.urdf.xacro (robot description, xacro)
@@ -51,6 +51,6 @@
           <samples>360</samples>
           <resolution>1</resolution>
-          <min_angle>-3.14159</min_angle>
-          <max_angle>3.14159</max_angle>
+          <min_angle>0.0</min_angle>
+          <max_angle>6.28319</max_angle>
         </horizontal>
       </scan>

File: kubot_description/urdf/model_xacro/kubot2.urdf.xacro (robot description, xacro)
@@ -14,10 +14,10 @@
 <xacro:property name="wheel_joint_z" value="0.080"/>
 <xacro:property name="caster_mass"    value="0.01"/>
-<xacro:property name="caster_radius"  value="0.015"/>
-<xacro:property name="caster_length"  value="0.02"/>
-<xacro:property name="caster_width"   value="0.3"/>
+<xacro:property name="caster_radius"  value="0.03"/>
+<xacro:property name="caster_length"  value="0.03"/>
+<xacro:property name="caster_width"   value="0.03"/>
 <xacro:property name="caster_joint_x" value="0.164"/>
 <xacro:property name="caster_joint_y" value="0.0"/>
-<xacro:property name="caster_joint_z" value="0.014"/>
+<xacro:property name="caster_joint_z" value="0.0165"/>
 <xacro:macro name="base">
 <!-- Robot Frame  a.k.a base_link -->
@@ -121,5 +121,5 @@
         <origin xyz="0 0 0" rpy="0 0 0"/>
         <geometry>
-            <sphere radius="${caster_radius}"/>
+                <box size="${caster_radius} ${caster_length} ${caster_width}"/>
         </geometry>
         <xacro:material_white/>
@@ -128,8 +128,18 @@
         <origin xyz="0 0 0" rpy="0 0 0"/>
         <geometry>
-                <sphere radius="${caster_radius}" />
+                <box size="${caster_radius} ${caster_length} ${caster_width}"/>
         </geometry>
     </collision>
-    <sphere_inertial_matrix  m="${caster_mass}" r="${caster_radius}" />
+    <inertial>
+        <origin xyz="0 0 0" rpy="0 0 0"/>
+        <mass value="${caster_mass}"/>
+        <inertia
+        ixx="0.001"
+        ixy="0.0"
+        ixz="0.0"
+        iyy="0.001"
+        iyz="0.0"
+        izz="0.001" />
+        </inertial>
     </link>
 <!-- Define Joint -->
@@ -145,5 +155,5 @@
         <parent link="base_link"/>
         <child link="wheel_right_link"/>
-        <origin xyz="0.0 ${-1*wheel_joint_y} ${wheel_joint_z}" rpy="0 0 ${M_PI}"/>
+        <origin xyz="${wheel_joint_x} ${-1*wheel_joint_y} ${wheel_joint_z}" rpy="0 0 ${M_PI}"/>
         <axis xyz="0 -1 0"/>
     </joint>
@@ -151,9 +161,9 @@
         <parent link="base_link"/>
         <child link="wheel_left_link"/>
-        <origin xyz="0.0 ${wheel_joint_y} ${wheel_joint_z}" rpy="0 0 0"/>
+        <origin xyz="${wheel_joint_x} ${wheel_joint_y} ${wheel_joint_z}" rpy="0 0 0"/>
         <axis xyz="0 1 0"/>
     </joint>
     <joint name="rear_caster_joint" type="fixed">
-        <origin xyz="${-1*caster_joint_x} 0 ${caster_joint_z}" rpy="0 0 0"/>
+        <origin xyz="${-1*caster_joint_x} ${caster_joint_y} ${caster_joint_z}" rpy="0 0 0"/>
         <parent link="base_link"/>
         <child link="rear_caster_link"/>
@@ -196,5 +206,4 @@
         <minDepth>0</minDepth>
         <maxVel>0.01</maxVel>
-        <fdir1>0 1 0</fdir1>
         <material>Gazebo/Black</material>
     </gazebo>
