Commit message: update

File: kubot_description/urdf/lidar_xacro/sick-tim551.urdf.xacro (robot description, xacro)
@@ -1,44 +1,75 @@
 <?xml version="1.0"?>
-<robot name="kubot" xmlns:xacro="https://ros.org/wiki/xacro">
-  <xacro:include filename="$(find kubot_description)/urdf/kubot_properties.urdf.xacro"/>
-  <xacro:macro
-  name="lidar"
-  params="frame:=laser_link lidar_enabled:=true lidar_joint_xyz:=0 lidar_joint_rpy:=0">
-      <xacro:if value="${lidar_enabled}">
-        <!-- laser link -->
-        <link name="${frame}">
-            <visual>
-                <origin xyz="0 0 -0.02" rpy="0 0 0"/>
-                <geometry>
-                    <mesh filename="package://kubot_description/meshes/lidar_frame/sick-tim551/laser_link.stl" scale="0.001 0.001 0.001"/>
-                </geometry>
-            <xacro:material_dark_grey/>
-            </visual>
-            <collision>
-                <origin xyz="0 0 -0.02" rpy="0 0 0"/>
-                <geometry>
-                    <mesh filename="package://kubot_description/meshes/lidar_frame/sick-tim551/laser_link.stl" scale="0.001 0.001 0.001"/>
-                </geometry>
-            <xacro:material_white/>
-            </collision>
-            <inertial>
-                <origin xyz="0 0 -0.02" rpy="0 0 0"/>
-                <mass value="0.195"/>
-                <inertia
-                   ixx="0.00028"
-                   ixy="0.0"
-                   ixz="0.0"
-                   iyy="0.00028"
-                   iyz="0.0"
-                   izz="0.00022" />
-            </inertial>
-        </link>
-        <!-- lidar joint -->
-        <joint name="lidar_joint" type="fixed">
-            <origin xyz="${lidar_joint_xyz}" rpy="${lidar_joint_rpy}" />
-            <parent link="base_link" />
-            <child link="${frame}" />
-        </joint>
-      </xacro:if>
-  </xacro:macro>
+<robot name="kubot_robot" xmlns:xacro="https://ros.org/wiki/xacro">
+<xacro:include filename="$(find kubot_description)/urdf/kubot_properties.urdf.xacro"/>
+<xacro:macro
+name="lidar"
+params="frame:=laser_link lidar_joint_xyz:=0 lidar_joint_rpy:=0">
+<!-- Laser Frame -->
+  <link name="${frame}">
+    <visual>
+      <origin xyz="0 0 -0.04" rpy="0 0 0"/>
+      <geometry>
+        <mesh filename="package://kubot_description/meshes/lidar_frame/$(arg lidar)/laser_link.stl" scale="0.001 0.001 0.001"/>
+      </geometry>
+      <xacro:material_dark_grey/>
+    </visual>
+    <collision>
+      <origin xyz="0 0 -0.04" rpy="0 0 0"/>
+      <geometry>
+        <cylinder length="0.03" radius="0.03"/>
+      </geometry>
+      <xacro:material_white/>
+    </collision>
+    <inertial>
+      <origin xyz="0 0 -0.04" rpy="0 0 0"/>
+      <mass value="0.179"/>
+      <inertia
+        ixx="0.001"
+        ixy="0.0"
+        ixz="0.0"
+        iyy="0.001"
+        iyz="0.0"
+        izz="0.001" />
+    </inertial>
+  </link>
+<!-- Define Joint -->
+  <joint name="lidar_joint" type="fixed">
+    <origin xyz="${lidar_joint_xyz}" rpy="${lidar_joint_rpy}" />
+    <parent link="base_link" />
+    <child link="${frame}" />
+  </joint>
+<!-- Define Gazebo -->
+  <gazebo reference="${frame}">
+    <material>Gazebo/DarkGrey</material>
+    <sensor type="ray" name="sick_tim551_sensor">
+    <pose>0 0 0 0 0 0</pose>
+    <visualize>1</visualize>
+    <update_rate>10</update_rate>
+    <ray>
+      <scan>
+        <horizontal>
+          <samples>360</samples>
+          <resolution>1</resolution>
+          <min_angle>-1.5708</min_angle>
+          <max_angle>1.5708</max_angle>
+        </horizontal>
+      </scan>
+      <range>
+        <min>0.08</min>
+        <max>15</max>
+        <resolution>0.01</resolution>
+      </range>
+      <noise>
+        <type>gaussian</type>
+        <mean>0.0</mean>
+        <stddev>0.004</stddev>
+      </noise>
+     </ray>
+     <plugin name="gazebo_ros_rplidar_controller" filename="libgazebo_ros_laser.so">
+        <topicName>scan</topicName>
+        <frameName>${frame}</frameName>
+     </plugin>
+     </sensor>
+  </gazebo>
+</xacro:macro>
 </robot>

File: kubot_description/urdf/model_xacro/kubot2.urdf.xacro (robot description, xacro)
@@ -46,4 +46,22 @@
         </inertial>
         </link>
+<!-- Logo Frame a.k.a adornment -->
+    <link name= "logo_frame">
+        <visual>
+            <origin xyz="0 0 0" rpy="0 0 0" />
+            <geometry>
+                <mesh filename="package://kubot_description/meshes/robot_frame/$(arg model)/logo_frame.stl" scale="0.001 0.001 0.001"/>
+            </geometry>
+            <xacro:material_white/>
+        </visual>
+        <collision>
+            <origin xyz="0 0 0" rpy="0 0 0" />
+            <geometry>
+                <mesh filename="package://kubot_description/meshes/robot_frame/$(arg model)/logo_frame.stl" scale="0.001 0.001 0.001"/>
+            </geometry>
+            <xacro:material_white/>
+        </collision>
+        <xacro:box_inertial_matrix m="0" a="0" b="0" c="0"/>
+    </link>
 <!-- Right Wheel Frame-->
     <link name= "wheel_right_link">
@@ -100,4 +118,8 @@
     </link>
 <!-- Define Joint -->
+    <joint name="logo_joint" type="fixed">
+        <parent link="base_link"/>
+        <child link="logo_frame"/>
+    </joint>
     <joint name="wheel_right_joint" type="continuous">
         <parent link="base_link"/>
@@ -120,4 +142,7 @@
     <gazebo reference="base_link">
         <material>Gazebo/Orange</material>
+    </gazebo>
+    <gazebo reference="logo_frame">
+        <material>Gazebo/White</material>
     </gazebo>
     <gazebo reference="wheel_right_link">

File: kubot_description/urdf/model_xacro/neuronbot2.urdf.xacro (robot description, xacro)
@@ -64,4 +64,22 @@
         <xacro:box_inertial_matrix m="0" a="0" b="0" c="0"/>
     </link>
+<!-- Logo Frame a.k.a adornment -->
+    <link name= "logo_frame">
+        <visual>
+            <origin xyz="0 0 0" rpy="0 0 0" />
+            <geometry>
+                <mesh filename="package://kubot_description/meshes/robot_frame/$(arg model)/logo_frame.stl" scale="0.001 0.001 0.001"/>
+            </geometry>
+            <xacro:material_red/>
+        </visual>
+        <collision>
+            <origin xyz="0 0 0" rpy="0 0 0" />
+            <geometry>
+                <mesh filename="package://kubot_description/meshes/robot_frame/$(arg model)/logo_frame.stl" scale="0.001 0.001 0.001"/>
+            </geometry>
+            <xacro:material_white/>
+        </collision>
+        <xacro:box_inertial_matrix m="0" a="0" b="0" c="0"/>
+    </link>
 <!-- Right Wheel Frame-->
     <link name= "wheel_right_link">
@@ -139,4 +157,8 @@
         <child link="r1_frame"/>
     </joint>
+    <joint name="logo_joint" type="fixed">
+        <parent link="base_link"/>
+        <child link="logo_frame"/>
+    </joint>
     <joint name="wheel_right_joint" type="continuous">
         <parent link="base_link"/>
@@ -166,4 +188,7 @@
     </gazebo>
     <gazebo reference="r1_frame">
+        <material>Gazebo/Red</material>
+    </gazebo>
+    <gazebo reference="logo_frame">
         <material>Gazebo/Red</material>
     </gazebo>

File: kubot_description/urdf/model_xacro/wagv.urdf.xacro (robot description, xacro)
@@ -1,111 +1,376 @@
 <?xml version="1.0"?>
-<robot name="kubot" xmlns:xacro="https://ros.org/wiki/xacro">
-  <xacro:include filename="$(find kubot_description)/urdf/kubot_properties.urdf.xacro"/>
-  <xacro:macro name="base">
-    <!-- Robot Frame  a.k.a base_link -->
+<robot name="kubot_robot" xmlns:xacro="https://ros.org/wiki/xacro">
+<xacro:include filename="$(find kubot_description)/urdf/kubot_properties.urdf.xacro"/>
+<xacro:property name="base_mass"    value="100"/>
+<xacro:property name="base_radius"  value="0.755"/>
+<xacro:property name="base_length"  value="0.675"/>
+<xacro:property name="base_width"   value="0.190"/>
+<xacro:property name="wheel_mass"    value="2"/>
+<xacro:property name="wheel_radius"  value="0.0770"/>
+<xacro:property name="wheel_length"  value="0.05"/>
+<xacro:property name="wheel_joint_x" value="0"/>
+<xacro:property name="wheel_joint_y" value="0.275"/>
+<xacro:property name="wheel_joint_z" value="0.075"/>
+<xacro:property name="caster_mass"    value="0.1"/>
+<xacro:property name="caster_radius"  value="0.029"/>
+<xacro:property name="caster_length"  value="0.05"/>
+<xacro:property name="caster_joint_x" value="0.268"/>
+<xacro:property name="caster_joint_y" value="0.185"/>
+<xacro:property name="caster_joint_z" value="0.028"/>
+<xacro:macro name="base">
+<!-- Robot Frame  a.k.a base_link -->
     <link name="base_link">
-        <visual name="visual_base">
-            <origin xyz="0 0 0" rpy="0 0 0" />
-            <geometry>
-                <mesh filename="package://kubot_description/meshes/robot_frame/wagv/base_link.stl" scale="0.001 0.001 0.001"/>
+        <visual>
+            <origin xyz="0 0 0" rpy="0 0 0" />
+            <geometry>
+                <mesh filename="package://kubot_description/meshes/robot_frame/$(arg model)/base_link.stl" scale="0.001 0.001 0.001"/>
             </geometry>
             <xacro:material_light_blue/>
         </visual>
         <collision>
-            <origin xyz="0 0 0" rpy="0 0 0" />
-            <geometry>
-                <mesh filename="package://kubot_description/meshes/robot_frame/wagv/base_link.stl" scale="0.001 0.001 0.001"/>
-            </geometry>
-            <xacro:material_white/>
+            <origin xyz="0 0 ${base_width/2+0.02}" rpy="0 0 0" />
+            <geometry>
+                <box size="${base_radius} ${base_length} ${base_width}"/>
+            </geometry>
         </collision>
         <inertial>
-          <origin xyz="0 0 0" rpy="0 0 0" />
-          <mass value="123.9982" />
-          <inertia
-              ixx="0.09617045"
-              ixy="3.5340082E-05"
-              ixz="2.5462637E-04"
-              iyy="0.1155512"
-              iyz="-4.2933341E-05"
-              izz="1.0718441E-01" />
-      </inertial>
-    </link>
-    <!-- r1_frame-->
+           <origin xyz=" 0 0 ${base_width/2+0.02} " rpy="0 0 0" />
+            <mass value="${base_mass}" />
+            <inertia
+            ixx="${base_mass*(base_length*base_length+base_width*base_width)/12}"
+            ixy = "0"
+            ixz = "0"
+            iyy="${base_mass*(base_radius*base_radius+base_width*base_width)/12}"
+            iyz = "0"
+            izz="${base_mass*(base_radius*base_radius+base_length*base_length)/12}" />
+        </inertial>
+        </link>
+<!-- R1 Frame a.k.a adornment -->
     <link name= "r1_frame">
         <visual>
             <origin xyz="0 0 0" rpy="0 0 0" />
             <geometry>
-                <mesh filename="package://kubot_description/meshes/robot_frame/wagv/r1_frame.stl" scale="0.001 0.001 0.001"/>
-            </geometry>
-            <xacro:material_white/>
-        </visual>
-    </link>
-    <!-- r2_frame-->
+                <mesh filename="package://kubot_description/meshes/robot_frame/$(arg model)/r1_frame.stl"/>
+            </geometry>
+            <xacro:material_white/>
+        </visual>
+        <collision>
+            <origin xyz="0 0 0" rpy="0 0 0" />
+            <geometry>
+                <mesh filename="package://kubot_description/meshes/robot_frame/$(arg model)/r1_frame.stl"/>
+            </geometry>
+            <xacro:material_white/>
+        </collision>
+        <xacro:box_inertial_matrix m="0" a="0" b="0" c="0"/>
+    </link>
+<!-- R2 Frame a.k.a adornment -->
     <link name= "r2_frame">
         <visual>
-            <origin xyz="0 0 0.05" rpy="0 0 0" />
-            <geometry>
-                <mesh filename="package://kubot_description/meshes/robot_frame/wagv/r2_frame.stl" scale="0.001 0.001 0.001"/>
+            <origin xyz="0 0 0" rpy="0 0 0" />
+            <geometry>
+                <mesh filename="package://kubot_description/meshes/robot_frame/$(arg model)/r2_frame.stl"/>
             </geometry>
             <xacro:material_dark_blue/>
         </visual>
-    </link>
-    <!-- Right Wheel_frame-->
+        <collision>
+            <origin xyz="0 0 0" rpy="0 0 0" />
+            <geometry>
+                <mesh filename="package://kubot_description/meshes/robot_frame/$(arg model)/r2_frame.stl"/>
+            </geometry>
+            <xacro:material_white/>
+        </collision>
+        <xacro:box_inertial_matrix m="0" a="0" b="0" c="0"/>
+    </link>
+<!-- R3 Frame a.k.a adornment -->
+    <link name= "r3_frame">
+        <visual>
+            <origin xyz="0 0 0" rpy="0 0 0" />
+            <geometry>
+                <mesh filename="package://kubot_description/meshes/robot_frame/$(arg model)/r3_frame.stl"/>
+            </geometry>
+            <xacro:material_black/>
+        </visual>
+        <collision>
+            <origin xyz="0 0 0" rpy="0 0 0" />
+            <geometry>
+                <mesh filename="package://kubot_description/meshes/robot_frame/$(arg model)/r3_frame.stl"/>
+            </geometry>
+            <xacro:material_white/>
+        </collision>
+        <xacro:box_inertial_matrix m="0" a="0" b="0" c="0"/>
+    </link>
+<!-- Logo Frame a.k.a adornment -->
+    <link name= "logo_frame">
+        <visual>
+            <origin xyz="0 0 0" rpy="0 0 0" />
+            <geometry>
+                <mesh filename="package://kubot_description/meshes/robot_frame/$(arg model)/logo_frame.stl"/>
+            </geometry>
+            <xacro:material_white/>
+        </visual>
+        <collision>
+            <origin xyz="0 0 0" rpy="0 0 0" />
+            <geometry>
+                <mesh filename="package://kubot_description/meshes/robot_frame/$(arg model)/logo_frame.stl"/>
+            </geometry>
+            <xacro:material_white/>
+        </collision>
+        <xacro:box_inertial_matrix m="0" a="0" b="0" c="0"/>
+    </link>
+<!-- Right Wheel Frame-->
     <link name= "wheel_right_link">
         <visual>
             <origin xyz="0 0 0" rpy="0 0 0" />
             <geometry>
-                <mesh filename="package://kubot_description/meshes/robot_frame/wagv/wheel_link.stl" scale="0.001 0.001 0.001"/>
-            </geometry>
-            <xacro:material_black/>
-        </visual>
-        <collision>
-              <origin xyz="0 0 0" rpy="0 0 0"/>
+                <mesh filename="package://kubot_description/meshes/robot_frame/$(arg model)/wheel_link.stl" scale="0.001 0.001 0.001"/>
+            </geometry>
+            <xacro:material_red/>
+        </visual>
+        <collision>
+              <origin xyz="0 0 0" rpy="${M_PI/2} 0 0"/>
               <geometry>
-                <mesh filename="package://kubot_description/meshes/robot_frame/wagv/wheel_link.stl" scale="0.001 0.001 0.001"/>
+                    <cylinder length="${wheel_length}" radius="${wheel_radius}"/>
               </geometry>
               <xacro:material_white/>
-         </collision>
-    </link>
-    <!-- Left Wheel_frame-->
+        </collision>
+        <xacro:cylinder_inertial_matrix m="${wheel_mass}" r="${wheel_radius}" h="${wheel_length}"/>
+    </link>
+<!-- Left Wheel Frame-->
     <link name= "wheel_left_link">
         <visual>
             <origin xyz="0 0 0" rpy="0 0 0" />
             <geometry>
-                <mesh filename="package://kubot_description/meshes/robot_frame/wagv/wheel_link.stl" scale="0.001 0.001 0.001"/>
-            </geometry>
-            <xacro:material_black/>
-        </visual>
-            <collision>
-              <origin xyz="0 0 0" rpy="0 0 0"/>
+                <mesh filename="package://kubot_description/meshes/robot_frame/$(arg model)/wheel_link.stl" scale="0.001 0.001 0.001"/>
+            </geometry>
+            <xacro:material_red/>
+        </visual>
+        <collision>
+              <origin xyz="0 0 0" rpy="${M_PI/2} 0 0"/>
               <geometry>
-                <mesh filename="package://kubot_description/meshes/robot_frame/wagv/wheel_link.stl" scale="0.001 0.001 0.001"/>
+                    <cylinder length="${wheel_length}" radius="${wheel_radius}"/>
               </geometry>
               <xacro:material_white/>
-         </collision>
-    </link>
-   <joint name="r1_joint" type="fixed">
-      <parent link="base_link"/>
-      <child link="r1_frame"/>
-   </joint>
+        </collision>
+        <xacro:cylinder_inertial_matrix m="${wheel_mass}" r="${wheel_radius}" h="${wheel_length}"/>
+    </link>
+<!-- Front Right Caster Frame -->
+    <link name="front_right_caster_link">
+    <visual>
+        <origin xyz="0 0 0" rpy="0 0 0"/>
+        <geometry>
+            <sphere radius="${caster_radius}"/>
+        </geometry>
+        <xacro:material_white/>
+    </visual>
+    <collision>
+        <origin xyz="0 0 0" rpy="0 0 0"/>
+        <geometry>
+                <sphere radius="${caster_radius}" />
+        </geometry>
+    </collision>
+    <sphere_inertial_matrix  m="${caster_mass}" r="${caster_radius}" />
+    </link>
+<!-- Front Left Caster Frame -->
+    <link name="front_left_caster_link">
+    <visual>
+        <origin xyz="0 0 0" rpy="0 0 0"/>
+        <geometry>
+            <sphere radius="${caster_radius}"/>
+        </geometry>
+        <xacro:material_white/>
+    </visual>
+    <collision>
+        <origin xyz="0 0 0" rpy="0 0 0"/>
+        <geometry>
+                <sphere radius="${caster_radius}" />
+        </geometry>
+    </collision>
+    <sphere_inertial_matrix  m="${caster_mass}" r="${caster_radius}" />
+    </link>
+<!-- Rear Right Caster Frame -->
+    <link name="rear_right_caster_link">
+    <visual>
+        <origin xyz="0 0 0" rpy="0 0 0"/>
+        <geometry>
+            <sphere radius="${caster_radius}"/>
+        </geometry>
+        <xacro:material_white/>
+    </visual>
+    <collision>
+        <origin xyz="0 0 0" rpy="0 0 0"/>
+        <geometry>
+                <sphere radius="${caster_radius}" />
+        </geometry>
+    </collision>
+    <sphere_inertial_matrix  m="${caster_mass}" r="${caster_radius}" />
+    </link>
+<!-- Rear Left Caster Frame -->
+    <link name="rear_left_caster_link">
+    <visual>
+        <origin xyz="0 0 0" rpy="0 0 0"/>
+        <geometry>
+            <sphere radius="${caster_radius}"/>
+        </geometry>
+        <xacro:material_white/>
+    </visual>
+    <collision>
+        <origin xyz="0 0 0" rpy="0 0 0"/>
+        <geometry>
+                <sphere radius="${caster_radius}" />
+        </geometry>
+    </collision>
+    <sphere_inertial_matrix  m="${caster_mass}" r="${caster_radius}" />
+    </link>
+<!-- Define Joint -->
+    <joint name="r1_joint" type="fixed">
+        <parent link="base_link"/>
+        <child link="r1_frame"/>
+    </joint>
    <joint name="r2_joint" type="fixed">
       <parent link="base_link"/>
       <child link="r2_frame"/>
    </joint>
-  <joint name="r_wheel_joint" type="continuous">
-    <parent link="base_link"/>
-    <child link="wheel_right_link"/>
-    <origin xyz="0.0 -0.275 0.07" rpy="0 0 0"/>
-    <axis xyz="0 -1 0"/>
-  </joint>
-  <joint name="l_wheel_joint" type="continuous">
-    <parent link="base_link"/>
-    <child link="wheel_left_link"/>
-    <origin xyz="0.0 0.275 0.07" rpy="0 0 0"/>
-    <axis xyz="0 1 0"/>
-  </joint>
+   <joint name="r3_joint" type="fixed">
+      <parent link="base_link"/>
+      <child link="r3_frame"/>
+   </joint>
+   <joint name="logo_joint" type="fixed">
+       <parent link="base_link"/>
+       <child link="logo_frame"/>
+   </joint>
+    <joint name="wheel_right_joint" type="continuous">
+        <parent link="base_link"/>
+        <child link="wheel_right_link"/>
+        <origin xyz="0.0 ${-1*wheel_joint_y} ${wheel_joint_z}" rpy="0 0 ${M_PI}"/>
+        <axis xyz="0 -1 0"/>
+    </joint>
+    <joint name="wheel_left_joint" type="continuous">
+        <parent link="base_link"/>
+        <child link="wheel_left_link"/>
+        <origin xyz="0.0 ${wheel_joint_y} ${wheel_joint_z}" rpy="0 0 0"/>
+        <axis xyz="0 1 0"/>
+    </joint>
+    <joint name="front_right_caster_joint" type="fixed">
+        <origin xyz="${caster_joint_x} ${caster_joint_y} ${caster_joint_z}" rpy="0 0 0"/>
+        <parent link="base_link"/>
+        <child link="front_right_caster_link"/>
+    </joint>
+    <joint name="front_left_caster_joint" type="fixed">
+        <origin xyz="${caster_joint_x} ${-1*caster_joint_y} ${caster_joint_z}" rpy="0 0 0"/>
+        <parent link="base_link"/>
+        <child link="front_left_caster_link"/>
+    </joint>
+    <joint name="rear_right_caster_joint" type="fixed">
+        <origin xyz="${-1*caster_joint_x} ${caster_joint_y} ${caster_joint_z}" rpy="0 0 0"/>
+        <parent link="base_link"/>
+        <child link="rear_right_caster_link"/>
+    </joint>
+    <joint name="rear_left_caster_joint" type="fixed">
+        <origin xyz="${-1*caster_joint_x} ${-1*caster_joint_y} ${caster_joint_z}" rpy="0 0 0"/>
+        <parent link="base_link"/>
+        <child link="rear_left_caster_link"/>
+    </joint>
+<!-- Define Gazebo -->
+    <gazebo reference="base_link">
+        <material>Gazebo/SkyBlue</material>
+    </gazebo>
+    <gazebo reference="r1_frame">
+        <material>Gazebo/White</material>
+    </gazebo>
+    <gazebo reference="r2_frame">
+        <material>Gazebo/Blue</material>
+    </gazebo>
+    <gazebo reference="r3_frame">
+        <material>Gazebo/Black</material>
+    </gazebo>
+    <gazebo reference="logo_frame">
+        <material>Gazebo/White</material>
+    </gazebo>
+    <gazebo reference="wheel_right_link">
+        <mu1>100000</mu1>
+        <mu2>100000</mu2>
+        <kp>500000.0</kp>
+        <kd>1.0</kd>
+        <minDepth>0.001</minDepth>
+        <maxVel>1.0</maxVel>
+        <fdir1>0 1 0</fdir1>
+        <material>Gazebo/Black</material>
+    </gazebo>
+    <gazebo reference="wheel_left_link">
+        <mu1>100000</mu1>
+        <mu2>100000</mu2>
+        <kp>500000.0</kp>
+        <kd>1.0</kd>
+        <minDepth>0.001</minDepth>
+        <maxVel>0.01</maxVel>
+        <fdir1>0 1 0</fdir1>
+        <material>Gazebo/Black</material>
+    </gazebo>
+    <gazebo reference="front_right_caster_link">
+        <mu1>0.1</mu1>
+        <mu2>0.1</mu2>
+        <kp>1000000.0</kp>
+        <kd>100.0</kd>
+        <minDepth>0</minDepth>
+        <maxVel>0.01</maxVel>
+        <fdir1>0 1 0</fdir1>
+        <material>Gazebo/Red</material>
+    </gazebo>
+    <gazebo reference="front_left_caster_link">
+        <mu1>0.1</mu1>
+        <mu2>0.1</mu2>
+        <kp>1000000.0</kp>
+        <kd>100.0</kd>
+        <minDepth>0</minDepth>
+        <maxVel>0.01</maxVel>
+        <fdir1>0 1 0</fdir1>
+        <material>Gazebo/Red</material>
+    </gazebo>
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