Commit message: add logi-c615

File: kubot_description/urdf/lidar_xacro/sick-tim551.urdf.xacro (robot description, xacro)
@@ -51,6 +51,6 @@
           <samples>360</samples>
           <resolution>1</resolution>
-          <min_angle>-1.5708</min_angle>
-          <max_angle>1.5708</max_angle>
+          <min_angle>-2.355</min_angle>
+          <max_angle>2.355</max_angle>
         </horizontal>
       </scan>

File: kubot_description/urdf/model_xacro/wagv.urdf.xacro (robot description, xacro)
@@ -24,5 +24,5 @@
             <origin xyz="0 0 0" rpy="0 0 0" />
             <geometry>
-                <mesh filename="package://kubot_description/meshes/robot_frame/$(arg model)/base_link.stl" scale="0.001 0.001 0.001"/>
+                <mesh filename="package://kubot_description/meshes/robot_frame/$(arg model)/base_link.stl"/>
             </geometry>
             <xacro:material_light_blue/>
@@ -74,7 +74,7 @@
         </visual>
         <collision>
-            <origin xyz="0 0 0" rpy="0 0 0" />
-            <geometry>
-                <mesh filename="package://kubot_description/meshes/robot_frame/$(arg model)/r2_frame.stl"/>
+            <origin xyz="0.005 0 0.27" rpy="0 0 0" />
+            <geometry>
+                <box size="0.5 0.64 0.1"/>
             </geometry>
             <xacro:material_white/>
@@ -375,5 +375,5 @@
 <xacro:property name="lidar_joint_rpy" value="0 0 0"/>
 <!-- Camera a.k.a Camera Pos -->
-<xacro:property name="camera_joint_xyz" value="0.26 0 0.17"/>
+<xacro:property name="camera_joint_xyz" value="0.355 0 0.130"/>
 <xacro:property name="camera_joint_rpy" value="0 0 0"/>
 </robot>
