Commit message: udpate

File: kubot_description/urdf/lidar_xacro/two-rplidar-a2.urdf.xacro (robot description, xacro)
@@ -8,5 +8,5 @@
   <link name="${frame}">
     <visual>
-        <origin xyz="0 0 0.031" rpy="0 0 0"/>
+        <origin xyz="0 0 0" rpy="0 0 0"/>
         <geometry>
             <mesh filename="package://kubot_description/meshes/lidar_frame/$(arg lidar)/laser_link.stl" scale="0.001 0.001 0.001"/>
@@ -15,12 +15,12 @@
     </visual>
     <collision>
-        <origin xyz="0 0 0.031" rpy="0 0 0"/>
-        <geometry>
-            <cylinder length="0.0515" radius="0.055"/>
+        <origin xyz="0 0 0" rpy="0 0 0"/>
+        <geometry>
+            <cylinder length="0.0415" radius="0.035"/>
         </geometry>
         <xacro:material_white/>
     </collision>
     <inertial>
-      <origin xyz="0 0 -0.0241" rpy="0 0 3.1415"/>
+      <origin xyz="0 0 0" rpy="0 0 3.1415"/>
       <mass value="0.179"/>
       <inertia
@@ -36,5 +36,5 @@
   <link name="lidar1_link">
     <visual>
-        <origin xyz="0 0 0.031" rpy="0 0 0"/>
+        <origin xyz="0 0 0" rpy="0 0 0"/>
         <geometry>
             <mesh filename="package://kubot_description/meshes/lidar_frame/$(arg lidar)/laser_link.stl" scale="0.001 0.001 0.001"/>
@@ -43,12 +43,12 @@
     </visual>
     <collision>
-        <origin xyz="0 0 0.031" rpy="0 0 0"/>
-        <geometry>
-            <cylinder length="0.0515" radius="0.055"/>
+        <origin xyz="0 0 0" rpy="0 0 0"/>
+        <geometry>
+            <cylinder length="0.0415" radius="0.035"/>
         </geometry>
         <xacro:material_white/>
     </collision>
     <inertial>
-      <origin xyz="0 0 -0.0241" rpy="0 0 3.1415"/>
+      <origin xyz="0 0 0" rpy="0 0 0"/>
       <mass value="0.179"/>
       <inertia
@@ -64,5 +64,5 @@
   <link name="lidar2_link">
     <visual>
-        <origin xyz="0 0 0.031" rpy="0 0 0"/>
+        <origin xyz="0 0 0" rpy="0 0 0"/>
         <geometry>
             <mesh filename="package://kubot_description/meshes/lidar_frame/$(arg lidar)/laser_link.stl" scale="0.001 0.001 0.001"/>
@@ -71,5 +71,5 @@
     </visual>
     <collision>
-        <origin xyz="0 0 0.031" rpy="0 0 0"/>
+        <origin xyz="0 0 0" rpy="0 0 0"/>
         <geometry>
             <cylinder length="0.0515" radius="0.055"/>
@@ -78,5 +78,5 @@
     </collision>
     <inertial>
-      <origin xyz="0 0 -0.0241" rpy="0 0 3.1415"/>
+      <origin xyz="0 0 0" rpy="0 0 0"/>
       <mass value="0.179"/>
       <inertia
@@ -96,10 +96,10 @@
   </joint>
   <joint name="lidar1_joint" type="fixed">
-    <origin xyz="0.319 0.208 0.166" rpy="0 0 0.7854" />
+    <origin xyz="0.319 0.208 0.197" rpy="0 0 0.7854" />
     <parent link="base_link" />
     <child link="lidar1_link" />
   </joint>
   <joint name="lidar2_joint" type="fixed">
-    <origin xyz="-0.319 -0.208 0.166" rpy="0 0 -2.355" />
+    <origin xyz="-0.319 -0.208 0.197" rpy="0 0 -2.355" />
     <parent link="base_link" />
     <child link="lidar2_link" />
@@ -154,5 +154,5 @@
       </scan>
       <range>
-        <min>0.15</min>
+        <min>0.12</min>
         <max>10</max>
         <resolution>0.01</resolution>
@@ -186,5 +186,5 @@
       </scan>
       <range>
-        <min>0.15</min>
+        <min>0.12</min>
         <max>10</max>
         <resolution>0.01</resolution>

File: kubot_description/urdf/model_xacro/aider.urdf.xacro (robot description, xacro)
@@ -1,108 +1,323 @@
 <?xml version="1.0"?>
-<robot name="kubot" xmlns:xacro="https://ros.org/wiki/xacro">
-  <xacro:include filename="$(find kubot_description)/urdf/kubot_properties.urdf.xacro"/>
-  <xacro:macro name="base">
-    <!-- Robot Frame  a.k.a base_link -->
+<robot name="kubot_robot" xmlns:xacro="https://ros.org/wiki/xacro">
+<xacro:include filename="$(find kubot_description)/urdf/kubot_properties.urdf.xacro"/>
+<xacro:property name="base_mass"    value="100"/>
+<xacro:property name="base_radius"  value="0.793"/>
+<xacro:property name="base_length"  value="0.530"/>
+<xacro:property name="base_width"   value="0.165"/>
+<xacro:property name="wheel_mass"    value="5"/>
+<xacro:property name="wheel_radius"  value="0.0755"/>
+<xacro:property name="wheel_length"  value="0.05"/>
+<xacro:property name="wheel_joint_x" value="0"/>
+<xacro:property name="wheel_joint_y" value="0.220"/>
+<xacro:property name="wheel_joint_z" value="0.075"/>
+<xacro:property name="caster_mass"    value="2"/>
+<xacro:property name="caster_radius"  value="0.0385"/>
+<xacro:property name="caster_length"  value="0.05"/>
+<xacro:property name="caster_joint_x" value="0.268"/>
+<xacro:property name="caster_joint_y" value="0.175"/>
+<xacro:property name="caster_joint_z" value="0.038"/>
+<xacro:macro name="base">
+<!-- Robot Frame  a.k.a base_link -->
     <link name="base_link">
-        <visual name="visual_base">
-            <origin xyz="0 0 0" rpy="0 0 0" />
-            <geometry>
-                <mesh filename="package://kubot_description/meshes/robot_frame/aider/base_link.stl" scale="0.001 0.001 0.001"/>
+        <visual>
+            <origin xyz="0 0 0" rpy="0 0 0" />
+            <geometry>
+                <mesh filename="package://kubot_description/meshes/robot_frame/$(arg model)/base_link.stl" scale="0.001 0.001 0.001"/>
             </geometry>
             <xacro:material_light_blue/>
         </visual>
         <collision>
-            <origin xyz="0 0 0" rpy="0 0 0" />
-            <geometry>
-                <mesh filename="package://kubot_description/meshes/robot_frame/aider/base_link.stl" scale="0.001 0.001 0.001"/>
+            <origin xyz="0 0 ${base_width/2+0.02}" rpy="0 0 0" />
+            <geometry>
+                <box size="${base_radius} ${base_length} ${base_width}"/>
+            </geometry>
+        </collision>
+        <inertial>
+           <origin xyz=" 0 0 ${base_width/2+0.02} " rpy="0 0 0" />
+            <mass value="${base_mass}" />
+            <inertia
+            ixx="${base_mass*(base_length*base_length+base_width*base_width)/12}"
+            ixy = "0"
+            ixz = "0"
+            iyy="${base_mass*(base_radius*base_radius+base_width*base_width)/12}"
+            iyz = "0"
+            izz="${base_mass*(base_radius*base_radius+base_length*base_length)/12}" />
+        </inertial>
+        </link>
+<!-- R1 Frame a.k.a adornment -->
+    <link name= "r1_frame">
+        <visual>
+            <origin xyz="0 0 0" rpy="0 0 0" />
+            <geometry>
+                <mesh filename="package://kubot_description/meshes/robot_frame/$(arg model)/r1_frame.stl" scale="0.001 0.001 0.001"/>
             </geometry>
             <xacro:material_white/>
-        </collision>
-        <inertial>
-          <origin xyz="0 0 0" rpy="0 0 0" />
-          <mass value="123.9982" />
-          <inertia
-              ixx="0.09617045"
-              ixy="3.5340082E-05"
-              ixz="2.5462637E-04"
-              iyy="0.1155512"
-              iyz="-4.2933341E-05"
-              izz="1.0718441E-01" />
-      </inertial>
-    </link>
-    <!-- r1_frame-->
-    <link name= "r1_frame">
-        <visual>
-            <origin xyz="0 0 0" rpy="0 0 0" />
-            <geometry>
-                <mesh filename="package://kubot_description/meshes/robot_frame/aider/r1_frame.stl" scale="0.001 0.001 0.001"/>
+        </visual>
+        <collision>
+            <origin xyz="0 0 0" rpy="0 0 0" />
+            <geometry>
+                <mesh filename="package://kubot_description/meshes/robot_frame/$(arg model)/r1_frame.stl" scale="0.001 0.001 0.001"/>
             </geometry>
             <xacro:material_white/>
-        </visual>
-    </link>
-    <!-- r2_frame-->
+        </collision>
+        <xacro:box_inertial_matrix m="0" a="0" b="0" c="0"/>
+    </link>
+<!-- R2 Frame a.k.a adornment -->
     <link name= "r2_frame">
         <visual>
             <origin xyz="0 0 0" rpy="0 0 0" />
             <geometry>
-                <mesh filename="package://kubot_description/meshes/robot_frame/aider/r2_frame.stl" scale="0.001 0.001 0.001"/>
+                <mesh filename="package://kubot_description/meshes/robot_frame/$(arg model)/r2_frame.stl" scale="0.001 0.001 0.001"/>
             </geometry>
             <xacro:material_dark_blue/>
         </visual>
-    </link>
-    <!-- Right Wheel_frame-->
+        <collision>
+            <origin xyz="0 0 0" rpy="0 0 0" />
+            <geometry>
+                <mesh filename="package://kubot_description/meshes/robot_frame/$(arg model)/r2_frame.stl" scale="0.001 0.001 0.001"/>
+            </geometry>
+            <xacro:material_white/>
+        </collision>
+        <xacro:box_inertial_matrix m="0" a="0" b="0" c="0"/>
+    </link>
+<!-- Right Wheel Frame-->
     <link name= "wheel_right_link">
         <visual>
             <origin xyz="0 0 0" rpy="0 0 0" />
             <geometry>
-                <mesh filename="package://kubot_description/meshes/robot_frame/aider/wheel_link.stl" scale="0.001 0.001 0.001"/>
+                <mesh filename="package://kubot_description/meshes/robot_frame/$(arg model)/wheel_link.stl" scale="0.001 0.001 0.001"/>
             </geometry>
             <xacro:material_black/>
         </visual>
         <collision>
-              <origin xyz="0 0 0" rpy="0 0 0"/>
+              <origin xyz="0 0 0" rpy="${M_PI/2} 0 0"/>
               <geometry>
-                <mesh filename="package://kubot_description/meshes/robot_frame/aider/wheel_link.stl" scale="0.001 0.001 0.001"/>
+                    <cylinder length="${wheel_length}" radius="${wheel_radius}"/>
               </geometry>
               <xacro:material_white/>
-         </collision>
-    </link>
-    <!-- Left Wheel_frame-->
+        </collision>
+        <xacro:cylinder_inertial_matrix m="${wheel_mass}" r="${wheel_radius}" h="${wheel_length}"/>
+    </link>
+<!-- Left Wheel Frame-->
     <link name= "wheel_left_link">
         <visual>
             <origin xyz="0 0 0" rpy="0 0 0" />
             <geometry>
-                <mesh filename="package://kubot_description/meshes/robot_frame/aider/wheel_link.stl" scale="0.001 0.001 0.001"/>
+                <mesh filename="package://kubot_description/meshes/robot_frame/$(arg model)/wheel_link.stl" scale="0.001 0.001 0.001"/>
             </geometry>
             <xacro:material_black/>
         </visual>
-            <collision>
-              <origin xyz="0 0 0" rpy="0 0 0"/>
+        <collision>
+              <origin xyz="0 0 0" rpy="${M_PI/2} 0 0"/>
               <geometry>
-                <mesh filename="package://kubot_description/meshes/robot_frame/aider/wheel_link.stl" scale="0.001 0.001 0.001"/>
+                    <cylinder length="${wheel_length}" radius="${wheel_radius}"/>
               </geometry>
               <xacro:material_white/>
-         </collision>
-    </link>
-   <joint name="r1_joint" type="fixed">
-      <parent link="base_link"/>
-      <child link="r1_frame"/>
-   </joint>
+        </collision>
+        <xacro:cylinder_inertial_matrix m="${wheel_mass}" r="${wheel_radius}" h="${wheel_length}"/>
+    </link>
+<!-- Front Right Caster Frame -->
+    <link name="front_right_caster_link">
+    <visual>
+        <origin xyz="0 0 0" rpy="0 0 0"/>
+        <geometry>
+            <sphere radius="${caster_radius}"/>
+        </geometry>
+        <xacro:material_white/>
+    </visual>
+    <collision>
+        <origin xyz="0 0 0" rpy="0 0 0"/>
+        <geometry>
+                <sphere radius="${caster_radius}" />
+        </geometry>
+    </collision>
+    <sphere_inertial_matrix  m="${caster_mass}" r="${caster_radius}" />
+    </link>
+<!-- Front Left Caster Frame -->
+    <link name="front_left_caster_link">
+    <visual>
+        <origin xyz="0 0 0" rpy="0 0 0"/>
+        <geometry>
+            <sphere radius="${caster_radius}"/>
+        </geometry>
+        <xacro:material_white/>
+    </visual>
+    <collision>
+        <origin xyz="0 0 0" rpy="0 0 0"/>
+        <geometry>
+                <sphere radius="${caster_radius}" />
+        </geometry>
+    </collision>
+    <sphere_inertial_matrix  m="${caster_mass}" r="${caster_radius}" />
+    </link>
+<!-- Rear Right Caster Frame -->
+    <link name="rear_right_caster_link">
+    <visual>
+        <origin xyz="0 0 0" rpy="0 0 0"/>
+        <geometry>
+            <sphere radius="${caster_radius}"/>
+        </geometry>
+        <xacro:material_white/>
+    </visual>
+    <collision>
+        <origin xyz="0 0 0" rpy="0 0 0"/>
+        <geometry>
+                <sphere radius="${caster_radius}" />
+        </geometry>
+    </collision>
+    <sphere_inertial_matrix  m="${caster_mass}" r="${caster_radius}" />
+    </link>
+<!-- Rear Left Caster Frame -->
+    <link name="rear_left_caster_link">
+    <visual>
+        <origin xyz="0 0 0" rpy="0 0 0"/>
+        <geometry>
+            <sphere radius="${caster_radius}"/>
+        </geometry>
+        <xacro:material_white/>
+    </visual>
+    <collision>
+        <origin xyz="0 0 0" rpy="0 0 0"/>
+        <geometry>
+                <sphere radius="${caster_radius}" />
+        </geometry>
+    </collision>
+    <sphere_inertial_matrix  m="${caster_mass}" r="${caster_radius}" />
+    </link>
+<!-- Define Joint -->
+    <joint name="r1_joint" type="fixed">
+        <parent link="base_link"/>
+        <child link="r1_frame"/>
+    </joint>
    <joint name="r2_joint" type="fixed">
       <parent link="base_link"/>
       <child link="r2_frame"/>
    </joint>
-  <joint name="r_wheel_joint" type="continuous">
-    <parent link="base_link"/>
-    <child link="wheel_right_link"/>
-    <origin xyz="0.0 0.2185 0.075" rpy="0 0 0"/>
-    <axis xyz="0 1 0"/>
-  </joint>
-  <joint name="l_wheel_joint" type="continuous">
-    <parent link="base_link"/>
-    <child link="wheel_left_link"/>
-    <origin xyz="0.0 -0.2185 0.075" rpy="0 0 3.14159"/>
-    <axis xyz="0 -1 0"/>
-  </joint>
+    <joint name="wheel_right_joint" type="continuous">
+        <parent link="base_link"/>
+        <child link="wheel_right_link"/>
+        <origin xyz="0.0 ${-1*wheel_joint_y} ${wheel_joint_z}" rpy="0 0 ${M_PI}"/>
+        <axis xyz="0 -1 0"/>
+    </joint>
+    <joint name="wheel_left_joint" type="continuous">
+        <parent link="base_link"/>
+        <child link="wheel_left_link"/>
+        <origin xyz="0.0 ${wheel_joint_y} ${wheel_joint_z}" rpy="0 0 0"/>
+        <axis xyz="0 1 0"/>
+    </joint>
+    <joint name="front_right_caster_joint" type="fixed">
+        <origin xyz="${caster_joint_x} ${caster_joint_y} ${caster_joint_z}" rpy="0 0 0"/>
+        <parent link="base_link"/>
+        <child link="front_right_caster_link"/>
+    </joint>
+    <joint name="front_left_caster_joint" type="fixed">
+        <origin xyz="${caster_joint_x} ${-1*caster_joint_y} ${caster_joint_z}" rpy="0 0 0"/>
+        <parent link="base_link"/>
+        <child link="front_left_caster_link"/>
+    </joint>
+    <joint name="rear_right_caster_joint" type="fixed">
+        <origin xyz="${-1*caster_joint_x} ${caster_joint_y} ${caster_joint_z}" rpy="0 0 0"/>
+        <parent link="base_link"/>
+        <child link="rear_right_caster_link"/>
+    </joint>
+    <joint name="rear_left_caster_joint" type="fixed">
+        <origin xyz="${-1*caster_joint_x} ${-1*caster_joint_y} ${caster_joint_z}" rpy="0 0 0"/>
+        <parent link="base_link"/>
+        <child link="rear_left_caster_link"/>
+    </joint>
+<!-- Define Gazebo -->
+    <gazebo reference="base_link">
+        <material>Gazebo/SkyBlue</material>
+    </gazebo>
+    <gazebo reference="r1_frame">
+        <material>Gazebo/White</material>
+    </gazebo>
+    <gazebo reference="r2_frame">
+        <material>Gazebo/Blue</material>
+    </gazebo>
+    <gazebo reference="wheel_right_link">
+        <mu1>100000</mu1>
+        <mu2>100000</mu2>
+        <kp>500000.0</kp>
+        <kd>1.0</kd>
+        <minDepth>0.001</minDepth>
+        <maxVel>1.0</maxVel>
+        <fdir1>0 1 0</fdir1>
+        <material>Gazebo/Black</material>
+    </gazebo>
+    <gazebo reference="wheel_left_link">
+        <mu1>100000</mu1>
+        <mu2>100000</mu2>
+        <kp>500000.0</kp>
+        <kd>1.0</kd>
+        <minDepth>0.001</minDepth>
+        <maxVel>0.01</maxVel>
+        <fdir1>0 1 0</fdir1>
+        <material>Gazebo/Black</material>
+    </gazebo>
+    <gazebo reference="front_right_caster_link">
+        <mu1>0.1</mu1>
+        <mu2>0.1</mu2>
+        <kp>1000000.0</kp>
+        <kd>100.0</kd>
+        <minDepth>0</minDepth>
+        <maxVel>0.01</maxVel>
+        <fdir1>0 1 0</fdir1>
+        <material>Gazebo/Red</material>
+    </gazebo>
+    <gazebo reference="front_left_caster_link">
+        <mu1>0.1</mu1>
+        <mu2>0.1</mu2>
+        <kp>1000000.0</kp>
+        <kd>100.0</kd>
+        <minDepth>0</minDepth>
+        <maxVel>0.01</maxVel>
+        <fdir1>0 1 0</fdir1>
+        <material>Gazebo/Red</material>
+    </gazebo>
+    <gazebo reference="rear_right_caster_link">
+        <mu1>0.1</mu1>
+        <mu2>0.1</mu2>
+        <kp>1000000.0</kp>
+        <kd>100.0</kd>
+        <minDepth>0</minDepth>
+        <maxVel>0.01</maxVel>
+        <fdir1>0 1 0</fdir1>
+        <material>Gazebo/Red</material>
+    </gazebo>
+    <gazebo reference="rear_left_caster_link">
+        <mu1>0.1</mu1>
+        <mu2>0.1</mu2>
+        <kp>1000000.0</kp>
+        <kd>100.0</kd>
+        <minDepth>0</minDepth>
+        <maxVel>0.01</maxVel>
+        <fdir1>0 1 0</fdir1>
+        <material>Gazebo/Red</material>
+    </gazebo>
+    <gazebo>
+        <plugin name="differential_drive_controller" filename="libgazebo_ros_diff_drive.so">
+            <commandTopic>cmd_vel</commandTopic>
+            <odometryTopic>odom</odometryTopic>
+            <odometryFrame>odom</odometryFrame>
+            <odometrySource>world</odometrySource>
+            <publishOdom>true</publishOdom>
+            <publishOdomTF>true</publishOdomTF>
+            <robotBaseFrame>footprint</robotBaseFrame>
+            <publishWheelTF>false</publishWheelTF>
+            <publishTf>true</publishTf>
+            <publishWheelJointState>true</publishWheelJointState>
+            <legacyMode>false</legacyMode>
+            <updateRate>30</updateRate>
+            <leftJoint>wheel_left_joint</leftJoint>
+            <rightJoint>wheel_right_joint</rightJoint>
+            <wheelSeparation>${wheel_joint_y*2}</wheelSeparation>
+            <wheelDiameter>${2*wheel_radius}</wheelDiameter>
+            <wheelAcceleration>1</wheelAcceleration>
+            <wheelTorque>10</wheelTorque>
+            <rosDebugLevel>na</rosDebugLevel>
+        </plugin>
+    </gazebo>
   </xacro:macro>
   <!-- Lidar Frame a.k.a Lidar Pos-->

Commit message: update aider robot urdf.xacro

File: kubot_description/urdf/lidar_xacro/two-rplidar-a2.urdf.xacro (robot description, xacro)
@@ -106,36 +106,4 @@
   </joint>
 <!-- Define Gazebo -->
-  <gazebo reference="${frame}">
-    <material>Gazebo/DarkGrey</material>
-    <sensor type="ray" name="rplidar_a2_ira_sensor">
-    <pose>0 0 0 0 0 0</pose>
-    <visualize>1</visualize>
-    <update_rate>5.5</update_rate>
-    <ray>
-      <scan>
-        <horizontal>
-          <samples>360</samples>
-          <resolution>1</resolution>
-          <min_angle>0.0</min_angle>
-          <max_angle>6.28319</max_angle>
-        </horizontal>
-      </scan>
-      <range>
-        <min>0.15</min>
-        <max>10</max>
-        <resolution>0.01</resolution>
-      </range>
-      <noise>
-        <type>gaussian</type>
-        <mean>0.0</mean>
-        <stddev>0.004</stddev>
-      </noise>
-     </ray>
-     <plugin name="gazebo_ros_rplidar_controller" filename="libgazebo_ros_laser.so">
-        <topicName>scan</topicName>
-        <frameName>${frame}</frameName>
-     </plugin>
-     </sensor>
-  </gazebo>
   <gazebo reference="lidar1_link">
     <material>Gazebo/DarkGrey</material>

File: kubot_description/urdf/model_xacro/aider.urdf.xacro (robot description, xacro)
@@ -6,16 +6,16 @@
 <xacro:property name="base_length"  value="0.530"/>
 <xacro:property name="base_width"   value="0.165"/>
-<xacro:property name="wheel_mass"    value="5"/>
-<xacro:property name="wheel_radius"  value="0.0755"/>
+<xacro:property name="wheel_mass"    value="0.5"/>
+<xacro:property name="wheel_radius"  value="0.0765"/>
 <xacro:property name="wheel_length"  value="0.05"/>
 <xacro:property name="wheel_joint_x" value="0"/>
 <xacro:property name="wheel_joint_y" value="0.220"/>
 <xacro:property name="wheel_joint_z" value="0.075"/>
-<xacro:property name="caster_mass"    value="0.01"/>
-<xacro:property name="caster_radius"  value="0.0385"/>
+<xacro:property name="caster_mass"    value="0.1"/>
+<xacro:property name="caster_radius"  value="0.029"/>
 <xacro:property name="caster_length"  value="0.05"/>
 <xacro:property name="caster_joint_x" value="0.268"/>
 <xacro:property name="caster_joint_y" value="0.175"/>
-<xacro:property name="caster_joint_z" value="0.038"/>
+<xacro:property name="caster_joint_z" value="0.028"/>
 <xacro:macro name="base">
 <!-- Robot Frame  a.k.a base_link -->

Commit message: update

File: kubot_description/urdf/lidar_xacro/two-rplidar-a2.urdf.xacro (robot description, xacro)
@@ -96,10 +96,10 @@
   </joint>
   <joint name="lidar1_joint" type="fixed">
-    <origin xyz="0.319 0.208 0.197" rpy="0 0 0.7854" />
+    <origin xyz="0.319 0.208 0.197" rpy="0 0 3.92699" />
     <parent link="base_link" />
     <child link="lidar1_link" />
   </joint>
   <joint name="lidar2_joint" type="fixed">
-    <origin xyz="-0.319 -0.208 0.197" rpy="0 0 -2.355" />
+    <origin xyz="-0.319 -0.208 0.197" rpy="0 0 -5.4966" />
     <parent link="base_link" />
     <child link="lidar2_link" />
