Commit message: update aider robot gazebo

File: kubot_description/urdf/lidar_xacro/two-rplidar-a2.urdf.xacro (robot description, xacro)
@@ -59,5 +59,5 @@
 				<origin xyz="0 0 0" rpy="0 0 0" />
 				<geometry>
-					<cylinder length="0.0515" radius="0.055" />
+					<cylinder length="0.0415" radius="0.035" />
 				</geometry>
 				<xacro:material_white />
@@ -76,10 +76,10 @@
 		</joint>
 		<joint name="lidar1_joint" type="fixed">
-			<origin xyz="0.319 0.208 0.197" rpy="0 0 3.92699" />
+			<origin xyz="0.358 0.225 0.197" rpy="0 0 3.92699" />
 			<parent link="base_link" />
 			<child link="lidar1_link" />
 		</joint>
 		<joint name="lidar2_joint" type="fixed">
-			<origin xyz="-0.319 -0.208 0.197" rpy="0 0 -5.4966" />
+			<origin xyz="-0.358 -0.225 0.197" rpy="0 0 -5.4966" />
 			<parent link="base_link" />
 			<child link="lidar2_link" />

File: kubot_description/urdf/model_xacro/aider.urdf.xacro (robot description, xacro)
@@ -3,17 +3,17 @@
     <xacro:include filename="$(find kubot_description)/urdf/kubot_properties.urdf.xacro" />
     <xacro:property name="base_mass" value="80" />
-    <xacro:property name="base_radius" value="0.793" />
-    <xacro:property name="base_length" value="0.530" />
-    <xacro:property name="base_width" value="0.165" />
+    <xacro:property name="base_radius" value="0.840" />
+    <xacro:property name="base_length" value="0.580" />
+    <xacro:property name="base_width" value="0.14" />
     <xacro:property name="wheel_mass" value="0.5" />
     <xacro:property name="wheel_radius" value="0.0765" />
     <xacro:property name="wheel_length" value="0.05" />
     <xacro:property name="wheel_joint_x" value="0" />
-    <xacro:property name="wheel_joint_y" value="0.220" />
+    <xacro:property name="wheel_joint_y" value="0.217" />
     <xacro:property name="wheel_joint_z" value="0.075" />
     <xacro:property name="caster_mass" value="0.1" />
     <xacro:property name="caster_radius" value="0.029" />
     <xacro:property name="caster_length" value="0.05" />
-    <xacro:property name="caster_joint_x" value="0.268" />
+    <xacro:property name="caster_joint_x" value="0.2473" />
     <xacro:property name="caster_joint_y" value="0.175" />
     <xacro:property name="caster_joint_z" value="0.028" />
@@ -49,11 +49,4 @@
                 <xacro:material_dark_blue />
             </visual>
-            <collision>
-                <origin xyz="0 0 0" rpy="0 0 0" />
-                <geometry>
-                    <mesh filename="package://kubot_description/meshes/robot_frame/$(arg model)/r1_frame.stl" scale="0.001 0.001 0.001" />
-                </geometry>
-            </collision>
-            <xacro:box_inertial_matrix m="0" a="0" b="0" c="0" />
         </link>
         <!-- R2 Frame a.k.a adornment -->
@@ -66,11 +59,4 @@
                 <xacro:material_black />
             </visual>
-            <collision>
-                <origin xyz="0 0 0" rpy="0 0 0" />
-                <geometry>
-                    <mesh filename="package://kubot_description/meshes/robot_frame/$(arg model)/r2_frame.stl" scale="0.001 0.001 0.001" />
-                </geometry>
-            </collision>
-            <xacro:box_inertial_matrix m="0" a="0" b="0" c="0" />
         </link>
         <!-- R3 Frame a.k.a adornment -->
@@ -83,11 +69,4 @@
                 <xacro:material_yellow />
             </visual>
-            <collision>
-                <origin xyz="0 0 0" rpy="0 0 0" />
-                <geometry>
-                    <mesh filename="package://kubot_description/meshes/robot_frame/$(arg model)/r3_frame.stl" scale="0.001 0.001 0.001" />
-                </geometry>
-            </collision>
-            <xacro:box_inertial_matrix m="0" a="0" b="0" c="0" />
         </link>
         <!-- Right Wheel Frame-->
@@ -107,5 +86,8 @@
                 <xacro:material_white />
             </collision>
-            <xacro:cylinder_inertial_matrix m="${wheel_mass}" r="${wheel_radius}" h="${wheel_length}" />
+			<inertial>
+				<origin xyz="0 ${-1*wheel_length/2} 0" rpy="${M_PI/2} 0 0" />
+				<xacro:cylinder_inertial_matrix m="${wheel_mass}" r="${wheel_radius}" h="${wheel_length}" />
+			</inertial>
         </link>
         <!-- Left Wheel Frame-->
@@ -125,5 +107,8 @@
                 <xacro:material_white />
             </collision>
-            <xacro:cylinder_inertial_matrix m="${wheel_mass}" r="${wheel_radius}" h="${wheel_length}" />
+			<inertial>
+				<origin xyz="0 ${-1*wheel_length/2} 0" rpy="${M_PI/2} 0 0" />
+				<xacro:cylinder_inertial_matrix m="${wheel_mass}" r="${wheel_radius}" h="${wheel_length}" />
+			</inertial>
         </link>
         <!-- Front Right Caster Frame -->

Commit message: udpate aider lidar

File: kubot_description/urdf/lidar_xacro/two-rplidar-a2.urdf.xacro (robot description, xacro)
@@ -76,10 +76,10 @@
 		</joint>
 		<joint name="lidar1_joint" type="fixed">
-			<origin xyz="0.358 0.225 0.197" rpy="0 0 3.92699" />
+			<origin xyz="0.359 0.23 0.197" rpy="0 0 3.92699" />
 			<parent link="base_link" />
 			<child link="lidar1_link" />
 		</joint>
 		<joint name="lidar2_joint" type="fixed">
-			<origin xyz="-0.358 -0.225 0.197" rpy="0 0 -5.4966" />
+			<origin xyz="-0.359 -0.23 0.197" rpy="0 0 -5.4966" />
 			<parent link="base_link" />
 			<child link="lidar2_link" />

Commit message: update two lidar param

File: kubot_description/urdf/lidar_xacro/two-rplidar-a2.urdf.xacro (robot description, xacro)
@@ -37,5 +37,5 @@
 				<origin xyz="0 0 0" rpy="0 0 0" />
 				<geometry>
-					<cylinder length="0.0415" radius="0.035" />
+					<cylinder length="0.0315" radius="0.035" />
 				</geometry>
 				<xacro:material_white />
@@ -59,5 +59,5 @@
 				<origin xyz="0 0 0" rpy="0 0 0" />
 				<geometry>
-					<cylinder length="0.0415" radius="0.035" />
+					<cylinder length="0.0315" radius="0.035" />
 				</geometry>
 				<xacro:material_white />
@@ -76,11 +76,11 @@
 		</joint>
 		<joint name="lidar1_joint" type="fixed">
-			<origin xyz="0.359 0.23 0.197" rpy="0 0 3.92699" />
-			<parent link="base_link" />
+			<origin xyz="0.357 0.233 -0.04" rpy="0 0 3.926990" />
+			<parent link="${frame}" />
 			<child link="lidar1_link" />
 		</joint>
 		<joint name="lidar2_joint" type="fixed">
-			<origin xyz="-0.359 -0.23 0.197" rpy="0 0 -5.4966" />
-			<parent link="base_link" />
+			<origin xyz="-0.357 -0.233 -0.04" rpy="0 0 0.785398" />
+			<parent link="${frame}" />
 			<child link="lidar2_link" />
 		</joint>

File: kubot_description/urdf/model_xacro/aider.urdf.xacro (robot description, xacro)
@@ -329,5 +329,5 @@
     </xacro:macro>
     <!-- Lidar Frame a.k.a Lidar Pos-->
-    <xacro:property name="lidar_joint_xyz" value="0 0 0.227" />
+    <xacro:property name="lidar_joint_xyz" value="0 0 0.237" />
     <xacro:property name="lidar_joint_rpy" value="0 0 0" />
     <!-- Camera a.k.a Camera Pos -->
