Commit message: udpate model

File: kubot_description/urdf/kubot_properties.urdf.xacro (robot description, xacro)
@@ -79,22 +79,14 @@
    <!-- Macro for inertia matrix -->
    <xacro:macro name="sphere_inertial_matrix" params="m r">
-      <inertial>
          <mass value="${m}" />
          <inertia ixx="${2*m*r*r/5}" ixy="0" ixz="0" iyy="${2*m*r*r/5}" iyz="0" izz="${2*m*r*r/5}" />
-      </inertial>
    </xacro:macro>
    <xacro:macro name="cylinder_inertial_matrix" params="m r h">
-      <inertial>
          <mass value="${m}" />
-         <inertia ixx="${m*(3*r*r+h*h)/12}" ixy="0" ixz="0" iyy="${m*r*r/2}" iyz="0" izz="${m*(3*r*r+h*h)/12}" />
-      </inertial>
+         <inertia ixx="${m*(3*r*r+h*h)/12}" ixy="0" ixz="0" iyy="${m*(3*r*r+h*h)/12}" iyz="0" izz="${m*r*r/2}" />
    </xacro:macro>
-   <!-- a, b,c a.k.a width, height, depth a.k.a x*, y*, z* -->
    <xacro:macro name="box_inertial_matrix" params="m a b c">
-      <inertial>
-         <origin xyz=" 0 0 ${c/2} " rpy="0 0 0" />
          <mass value="${m}" />
          <inertia ixx="${m*(b*b+c*c)/12}" ixy="0" ixz="0" iyy="${m*(a*a+c*c)/12}" iyz="0" izz="${m*(a*a+b*b)/12}" />
-      </inertial>
    </xacro:macro>
 </robot>

File: kubot_description/urdf/model_xacro/aider.urdf.xacro (robot description, xacro)
@@ -127,5 +127,5 @@
                 </geometry>
             </collision>
-            <sphere_inertial_matrix m="${caster_mass}" r="${caster_radius}" />
+            <xacro:sphere_inertial_matrix m="${caster_mass}" r="${caster_radius}" />
         </link>
         <!-- Front Left Caster Frame -->
@@ -144,5 +144,5 @@
                 </geometry>
             </collision>
-            <sphere_inertial_matrix m="${caster_mass}" r="${caster_radius}" />
+            <xacro:sphere_inertial_matrix m="${caster_mass}" r="${caster_radius}" />
         </link>
         <!-- Rear Right Caster Frame -->
@@ -161,5 +161,5 @@
                 </geometry>
             </collision>
-            <sphere_inertial_matrix m="${caster_mass}" r="${caster_radius}" />
+            <xacro:sphere_inertial_matrix m="${caster_mass}" r="${caster_radius}" />
         </link>
         <!-- Rear Left Caster Frame -->
@@ -178,5 +178,5 @@
                 </geometry>
             </collision>
-            <sphere_inertial_matrix m="${caster_mass}" r="${caster_radius}" />
+            <xacro:sphere_inertial_matrix m="${caster_mass}" r="${caster_radius}" />
         </link>
         <!-- Define Joint -->

File: kubot_description/urdf/model_xacro/kubot2.urdf.xacro (robot description, xacro)
@@ -1,4 +1,5 @@
 <?xml version="1.0"?>
-<robot name="kubot_robot" xmlns:xacro="https://ros.org/wiki/xacro">
+<robot name="kubot_robot"
+	xmlns:xacro="https://ros.org/wiki/xacro">
 	<xacro:include filename="$(find kubot_description)/urdf/kubot_properties.urdf.xacro" />
 	<xacro:property name="base_mass" value="4.2" />
@@ -6,5 +7,5 @@
 	<xacro:property name="base_length" value="0.320" />
 	<xacro:property name="base_width" value="0.145" />
-	<xacro:property name="wheel_mass" value="0.05" />
+	<xacro:property name="wheel_mass" value="0.1" />
 	<xacro:property name="wheel_radius" value="0.0815" />
 	<xacro:property name="wheel_length" value="0.020" />
@@ -13,5 +14,5 @@
 	<xacro:property name="wheel_joint_y" value="0.122" />
 	<xacro:property name="wheel_joint_z" value="0.080" />
-	<xacro:property name="caster_mass" value="0.01" />
+	<xacro:property name="caster_mass" value="0.05" />
 	<xacro:property name="caster_radius" value="0.03" />
 	<xacro:property name="caster_length" value="0.03" />
@@ -19,5 +20,5 @@
 	<xacro:property name="caster_joint_x" value="0.164" />
 	<xacro:property name="caster_joint_y" value="0.0" />
-	<xacro:property name="caster_joint_z" value="0.0165" />
+	<xacro:property name="caster_joint_z" value="0.015" />
 	<xacro:macro name="base">
 		<!-- Robot Frame  a.k.a base_link -->
@@ -38,6 +39,5 @@
 			<inertial>
 				<origin xyz="-0.05 0 ${base_width/2+0.02} " rpy="0 0 0" />
-				<mass value="${base_mass}" />
-				<inertia ixx="${base_mass*(base_length*base_length+base_width*base_width)/12}" ixy="0" ixz="0" iyy="${base_mass*(base_radius*base_radius+base_width*base_width)/12}" iyz="0" izz="${base_mass*(base_radius*base_radius+base_length*base_length)/12}" />
+				<xacro:box_inertial_matrix m="${base_mass}" a="${base_radius}" b="${base_length}" c="${base_width}" />
 			</inertial>
 		</link>
@@ -51,11 +51,8 @@
 				<xacro:material_orange />
 			</visual>
-			<collision>
-				<origin xyz="0 0 0" rpy="0 0 0" />
-				<geometry>
-					<box size="0.0001 0.0001 0.0001" />
-				</geometry>
-			</collision>
-			<xacro:box_inertial_matrix m="0" a="0" b="0" c="0" />
+			<inertial>
+				<origin xyz="0 0 0" rpy="0 0 0" />
+				<xacro:box_inertial_matrix m="0.001" a="0.001" b="0.001" c="0.001" />
+			</inertial>
 		</link>
 		<!-- Logo Frame a.k.a adornment -->
@@ -68,11 +65,8 @@
 				<xacro:material_white />
 			</visual>
-			<collision>
-				<origin xyz="0 0 0" rpy="0 0 0" />
-				<geometry>
-					<box size="0.0001 0.0001 0.0001" />
-				</geometry>
-			</collision>
-			<xacro:box_inertial_matrix m="0" a="0" b="0" c="0" />
+			<inertial>
+				<origin xyz="0 0 0" rpy="0 0 0" />
+				<xacro:box_inertial_matrix m="0.001" a="0.001" b="0.001" c="0.001" />
+			</inertial>
 		</link>
 		<!-- Right Wheel Frame-->
@@ -91,5 +85,8 @@
 				</geometry>
 			</collision>
-			<xacro:cylinder_inertial_matrix m="${wheel_mass}" r="${wheel_radius}" h="${wheel_length}" />
+			<inertial>
+				<origin xyz="0 0 0" rpy="${M_PI/2} 0 0" />
+				<xacro:cylinder_inertial_matrix m="${wheel_mass}" r="${wheel_radius}" h="${wheel_length}" />
+			</inertial>
 		</link>
 		<!-- Left Wheel Frame-->
@@ -108,5 +105,8 @@
 				</geometry>
 			</collision>
-			<xacro:cylinder_inertial_matrix m="${wheel_mass}" r="${wheel_radius}" h="${wheel_length}" />
+			<inertial>
+				<origin xyz="0 0 0" rpy="${M_PI/2} 0 0" />
+				<xacro:cylinder_inertial_matrix m="${wheel_mass}" r="${wheel_radius}" h="${wheel_length}" />
+			</inertial>
 		</link>
 		<!-- Rear Caster Frame -->
@@ -127,6 +127,5 @@
 			<inertial>
 				<origin xyz="0 0 0" rpy="0 0 0" />
-				<mass value="${caster_mass}" />
-				<inertia ixx="0.001" ixy="0.0" ixz="0.0" iyy="0.001" iyz="0.0" izz="0.001" />
+				<xacro:sphere_inertial_matrix m="${caster_mass}" r="${caster_radius}" />
 			</inertial>
 		</link>

File: kubot_description/urdf/model_xacro/neuronbot2.urdf.xacro (robot description, xacro)
@@ -1,4 +1,5 @@
 <?xml version="1.0"?>
-<robot name="kubot_robot" xmlns:xacro="https://ros.org/wiki/xacro">
+<robot name="kubot_robot"
+	xmlns:xacro="https://ros.org/wiki/xacro">
 	<xacro:include filename="$(find kubot_description)/urdf/kubot_properties.urdf.xacro" />
 	<xacro:property name="base_mass" value="8.3" />
@@ -6,5 +7,5 @@
 	<xacro:property name="base_length" value="0.265" />
 	<xacro:property name="base_width" value="0.200" />
-	<xacro:property name="wheel_mass" value="0.05" />
+	<xacro:property name="wheel_mass" value="0.1" />
 	<xacro:property name="wheel_radius" value="0.042" />
 	<xacro:property name="wheel_length" value="0.02" />
@@ -12,10 +13,11 @@
 	<xacro:property name="wheel_joint_y" value="0.125" />
 	<xacro:property name="wheel_joint_z" value="0.041" />
-	<xacro:property name="caster_mass" value="0.01" />
-	<xacro:property name="caster_radius" value="0.015" />
-	<xacro:property name="caster_length" value="0.02" />
+	<xacro:property name="caster_mass" value="0.05" />
+	<xacro:property name="caster_radius" value="0.03" />
+	<xacro:property name="caster_length" value="0.03" />
+	<xacro:property name="caster_width" value="0.03" />
 	<xacro:property name="caster_joint_x" value="0.09" />
-	<xacro:property name="caster_joint_y" value="0.07" />
-	<xacro:property name="caster_joint_z" value="0.014" />
+	<xacro:property name="caster_joint_y" value="0" />
+	<xacro:property name="caster_joint_z" value="0.015" />
 	<xacro:macro name="base">
 		<!-- Robot Frame  a.k.a base_link -->
@@ -35,7 +37,6 @@
 			</collision>
 			<inertial>
-				<origin xyz=" 0 0 ${base_width/2+0.02} " rpy="0 0 0" />
-				<mass value="${base_mass}" />
-				<inertia ixx="${base_mass*(base_length*base_length+base_width*base_width)/12}" ixy="0" ixz="0" iyy="${base_mass*(base_radius*base_radius+base_width*base_width)/12}" iyz="0" izz="${base_mass*(base_radius*base_radius+base_length*base_length)/12}" />
+				<origin xyz="0 0 ${base_width/2+0.02} " rpy="0 0 0" />
+				<xacro:box_inertial_matrix m="${base_mass}" a="${base_radius}" b="${base_length}" c="${base_width}" />
 			</inertial>
 		</link>
@@ -49,11 +50,8 @@
 				<xacro:material_red />
 			</visual>
-			<collision>
-				<origin xyz="0 0 0" rpy="0 0 0" />
-				<geometry>
-					<box size="0.0001 0.0001 0.0001" />
-				</geometry>
-			</collision>
-			<xacro:box_inertial_matrix m="0" a="0" b="0" c="0" />
+			<inertial>
+				<origin xyz="0 0 0" rpy="0 0 0" />
+				<xacro:box_inertial_matrix m="0.001" a="0.001" b="0.001" c="0.001" />
+			</inertial>
 		</link>
 		<!-- Logo Frame a.k.a adornment -->
@@ -66,11 +64,8 @@
 				<xacro:material_red />
 			</visual>
-			<collision>
-				<origin xyz="0 0 0" rpy="0 0 0" />
-				<geometry>
-					<box size="0.0001 0.0001 0.0001" />
-				</geometry>
-			</collision>
-			<xacro:box_inertial_matrix m="0" a="0" b="0" c="0" />
+			<inertial>
+				<origin xyz="0 0 0" rpy="0 0 0" />
+				<xacro:box_inertial_matrix m="0.001" a="0.001" b="0.001" c="0.001" />
+			</inertial>
 		</link>
 		<!-- Right Wheel Frame-->
@@ -89,5 +84,8 @@
 				</geometry>
 			</collision>
-			<xacro:cylinder_inertial_matrix m="${wheel_mass}" r="${wheel_radius}" h="${wheel_length}" />
+			<inertial>
+				<origin xyz="0 ${-1*wheel_length/2} 0" rpy="${M_PI/2} 0 0" />
+				<xacro:cylinder_inertial_matrix m="${wheel_mass}" r="${wheel_radius}" h="${wheel_length}" />
+			</inertial>
 		</link>
 		<!-- Left Wheel Frame-->
@@ -107,5 +105,8 @@
 				<xacro:material_white />
 			</collision>
-			<xacro:cylinder_inertial_matrix m="${wheel_mass}" r="${wheel_radius}" h="${wheel_length}" />
+			<inertial>
+				<origin xyz="0 ${-1*wheel_length/2} 0" rpy="${M_PI/2} 0 0" />
+				<xacro:cylinder_inertial_matrix m="${wheel_mass}" r="${wheel_radius}" h="${wheel_length}" />
+			</inertial>
 		</link>
 		<!-- Front Caster Frame -->
@@ -114,5 +115,5 @@
 				<origin xyz="0 0 0" rpy="0 0 0" />
 				<geometry>
-					<sphere radius="${caster_radius}" />
+					<box size="${caster_radius} ${caster_length} ${caster_width}" />
 				</geometry>
 				<xacro:material_white />
@@ -121,8 +122,11 @@
 				<origin xyz="0 0 0" rpy="0 0 0" />
 				<geometry>
-					<sphere radius="${caster_radius}" />
-				</geometry>
-			</collision>
-			<sphere_inertial_matrix m="${caster_mass}" r="${caster_radius}" />
+					<box size="${caster_radius} ${caster_length} ${caster_width}" />
+				</geometry>
+			</collision>
+			<inertial>
+				<origin xyz="0 0 0" rpy="0 0 0" />
+				<xacro:sphere_inertial_matrix m="${caster_mass}" r="${caster_radius}" />
+			</inertial>
 		</link>
 		<!-- Rear Caster Frame -->
@@ -131,5 +135,5 @@
 				<origin xyz="0 0 0" rpy="0 0 0" />
 				<geometry>
-					<sphere radius="${caster_radius}" />
+					<box size="${caster_radius} ${caster_length} ${caster_width}" />
 				</geometry>
 				<xacro:material_white />
@@ -138,8 +142,11 @@
 				<origin xyz="0 0 0" rpy="0 0 0" />
 				<geometry>
-					<sphere radius="${caster_radius}" />
-				</geometry>
-			</collision>
-			<sphere_inertial_matrix m="${caster_mass}" r="${caster_radius}" />
+					<box size="${caster_radius} ${caster_length} ${caster_width}" />
+				</geometry>
+			</collision>
+			<inertial>
+				<origin xyz="0 0 0" rpy="0 0 0" />
+				<xacro:sphere_inertial_matrix m="${caster_mass}" r="${caster_radius}" />
+			</inertial>
 		</link>
 		<!-- Define Joint -->
@@ -165,10 +172,10 @@
 		</joint>
 		<joint name="front_caster_joint" type="fixed">
-			<origin xyz="${caster_joint_x} 0 ${caster_joint_z}" rpy="0 0 0" />
+			<origin xyz="${caster_joint_x} ${caster_joint_y} ${caster_joint_z}" rpy="0 0 0" />
 			<parent link="base_link" />
 			<child link="front_caster_link" />
 		</joint>
 		<joint name="rear_caster_joint" type="fixed">
-			<origin xyz="${-1*caster_joint_x} 0 ${caster_joint_z}" rpy="0 0 0" />
+			<origin xyz="${-1*caster_joint_x} ${caster_joint_y} ${caster_joint_z}" rpy="0 0 0" />
 			<parent link="base_link" />
 			<child link="rear_caster_link" />
@@ -211,5 +218,4 @@
 			<minDepth>0</minDepth>
 			<maxVel>0.01</maxVel>
-			<fdir1>0 1 0</fdir1>
 			<material>Gazebo/Black</material>
 		</gazebo>
@@ -221,5 +227,4 @@
 			<minDepth>0</minDepth>
 			<maxVel>0.01</maxVel>
-			<fdir1>0 1 0</fdir1>
 			<material>Gazebo/Black</material>
 		</gazebo>

File: kubot_description/urdf/model_xacro/wagv.urdf.xacro (robot description, xacro)
@@ -6,5 +6,5 @@
 	<xacro:property name="base_length" value="0.675" />
 	<xacro:property name="base_width" value="0.200" />
-	<xacro:property name="wheel_mass" value="0.5" />
+	<xacro:property name="wheel_mass" value="2" />
 	<xacro:property name="wheel_radius" value="0.0765" />
 	<xacro:property name="wheel_length" value="0.05" />
@@ -12,10 +12,11 @@
 	<xacro:property name="wheel_joint_y" value="0.280" />
 	<xacro:property name="wheel_joint_z" value="0.075" />
-	<xacro:property name="caster_mass" value="0.1" />
-	<xacro:property name="caster_radius" value="0.029" />
-	<xacro:property name="caster_length" value="0.05" />
+	<xacro:property name="caster_mass" value="1" />
+	<xacro:property name="caster_radius" value="0.03" />
+	<xacro:property name="caster_length" value="0.03" />
+	<xacro:property name="caster_width" value="0.03" />
 	<xacro:property name="caster_joint_x" value="0.268" />
 	<xacro:property name="caster_joint_y" value="0.175" />
-	<xacro:property name="caster_joint_z" value="0.028" />
+	<xacro:property name="caster_joint_z" value="0.015" />
 	<xacro:macro name="base">
 		<!-- Robot Frame  a.k.a base_link -->
@@ -36,6 +37,5 @@
 			<inertial>
 				<origin xyz=" 0 0 ${base_width/2+0.02} " rpy="0 0 0" />
-				<mass value="${base_mass}" />
-				<inertia ixx="${base_mass*(base_length*base_length+base_width*base_width)/12}" ixy="0" ixz="0" iyy="${base_mass*(base_radius*base_radius+base_width*base_width)/12}" iyz="0" izz="${base_mass*(base_radius*base_radius+base_length*base_length)/12}" />
+				<xacro:box_inertial_matrix m="${base_mass}" a="${base_radius}" b="${base_length}" c="${base_width}" />
 			</inertial>
 		</link>
@@ -49,12 +49,8 @@
 				<xacro:material_white />
 			</visual>
-			<collision>
-				<origin xyz="0 0 0" rpy="0 0 0" />
-				<geometry>
-					<mesh filename="package://kubot_description/meshes/robot_frame/$(arg model)/r1_frame.stl" />
-				</geometry>
-				<xacro:material_white />
-			</collision>
-			<xacro:box_inertial_matrix m="0" a="0" b="0" c="0" />
+			<inertial>
+				<origin xyz="0 0 0" rpy="0 0 0" />
+				<xacro:box_inertial_matrix m="0.001" a="0.001" b="0.001" c="0.001" />
+			</inertial>
 		</link>
 		<!-- R2 Frame a.k.a adornment -->
@@ -74,5 +70,8 @@
 				<xacro:material_white />
 			</collision>
-			<xacro:box_inertial_matrix m="0" a="0" b="0" c="0" />
+			<inertial>
+				<origin xyz="0 0 0" rpy="0 0 0" />
+				<xacro:box_inertial_matrix m="0.001" a="0.001" b="0.001" c="0.001" />
+			</inertial>
 		</link>
 		<!-- R3 Frame a.k.a adornment -->
@@ -85,12 +84,8 @@
 				<xacro:material_black />
 			</visual>
-			<collision>
-				<origin xyz="0 0 0" rpy="0 0 0" />
-				<geometry>
-					<mesh filename="package://kubot_description/meshes/robot_frame/$(arg model)/r3_frame.stl" />
-				</geometry>
-				<xacro:material_white />
-			</collision>
-			<xacro:box_inertial_matrix m="0" a="0" b="0" c="0" />
+			<inertial>
+				<origin xyz="0 0 0" rpy="0 0 0" />
+				<xacro:box_inertial_matrix m="0.001" a="0.001" b="0.001" c="0.001" />
+			</inertial>
 		</link>
 		<!-- Logo Frame a.k.a adornment -->
@@ -103,12 +98,8 @@
 				<xacro:material_white />
 			</visual>
-			<collision>
-				<origin xyz="0 0 0" rpy="0 0 0" />
-				<geometry>
-					<mesh filename="package://kubot_description/meshes/robot_frame/$(arg model)/logo_frame.stl" />
-				</geometry>
-				<xacro:material_white />
-			</collision>
-			<xacro:box_inertial_matrix m="0" a="0" b="0" c="0" />
+			<inertial>
+				<origin xyz="0 0 0" rpy="0 0 0" />
+				<xacro:box_inertial_matrix m="0.001" a="0.001" b="0.001" c="0.001" />
+			</inertial>
 		</link>
 		<!-- Right Wheel Frame-->
@@ -126,7 +117,9 @@
 					<cylinder length="${wheel_length}" radius="${wheel_radius}" />
 				</geometry>
-				<xacro:material_white />
-			</collision>
-			<xacro:cylinder_inertial_matrix m="${wheel_mass}" r="${wheel_radius}" h="${wheel_length}" />
+			</collision>
+			<inertial>
+				<origin xyz="0 0 0" rpy="${M_PI/2} 0 0" />
+				<xacro:cylinder_inertial_matrix m="${wheel_mass}" r="${wheel_radius}" h="${wheel_length}" />
+			</inertial>
 		</link>
 		<!-- Left Wheel Frame-->
@@ -146,5 +139,8 @@
 				<xacro:material_white />
 			</collision>
-			<xacro:cylinder_inertial_matrix m="${wheel_mass}" r="${wheel_radius}" h="${wheel_length}" />
+			<inertial>
+				<origin xyz="0 0 0" rpy="${M_PI/2} 0 0" />
+				<xacro:cylinder_inertial_matrix m="${wheel_mass}" r="${wheel_radius}" h="${wheel_length}" />
+			</inertial>
 		</link>
 		<!-- Front Right Caster Frame -->
@@ -160,8 +156,11 @@
 				<origin xyz="0 0 0" rpy="0 0 0" />
 				<geometry>
-					<sphere radius="${caster_radius}" />
-				</geometry>
-			</collision>
-			<sphere_inertial_matrix m="${caster_mass}" r="${caster_radius}" />
+					<box size="${caster_radius} ${caster_length} ${caster_width}" />
+				</geometry>
+			</collision>
+			<inertial>
+				<origin xyz="0 0 0" rpy="0 0 0" />
+				<xacro:sphere_inertial_matrix m="${caster_mass}" r="${caster_radius}" />
+			</inertial>
 		</link>
 		<!-- Front Left Caster Frame -->
@@ -177,8 +176,11 @@
 				<origin xyz="0 0 0" rpy="0 0 0" />
 				<geometry>
-					<sphere radius="${caster_radius}" />
-				</geometry>
-			</collision>
-			<sphere_inertial_matrix m="${caster_mass}" r="${caster_radius}" />
+					<box size="${caster_radius} ${caster_length} ${caster_width}" />
+				</geometry>
+			</collision>
+			<inertial>
+				<origin xyz="0 0 0" rpy="0 0 0" />
+				<xacro:sphere_inertial_matrix m="${caster_mass}" r="${caster_radius}" />
+			</inertial>
 		</link>
 		<!-- Rear Right Caster Frame -->
@@ -194,8 +196,11 @@
 				<origin xyz="0 0 0" rpy="0 0 0" />
 				<geometry>
-					<sphere radius="${caster_radius}" />
-				</geometry>
-			</collision>
-			<sphere_inertial_matrix m="${caster_mass}" r="${caster_radius}" />
+					<box size="${caster_radius} ${caster_length} ${caster_width}" />
+				</geometry>
+			</collision>
+			<inertial>
+				<origin xyz="0 0 0" rpy="0 0 0" />
+				<xacro:sphere_inertial_matrix m="${caster_mass}" r="${caster_radius}" />
+			</inertial>
 		</link>
 		<!-- Rear Left Caster Frame -->
@@ -211,8 +216,11 @@
 				<origin xyz="0 0 0" rpy="0 0 0" />
 				<geometry>
-					<sphere radius="${caster_radius}" />
-				</geometry>
-			</collision>
-			<sphere_inertial_matrix m="${caster_mass}" r="${caster_radius}" />
+					<box size="${caster_radius} ${caster_length} ${caster_width}" />
+				</geometry>
+			</collision>
+			<inertial>
+				<origin xyz="0 0 0" rpy="0 0 0" />
+				<xacro:sphere_inertial_matrix m="${caster_mass}" r="${caster_radius}" />
+			</inertial>
 		</link>
 		<!-- Define Joint -->
@@ -236,5 +244,5 @@
 			<parent link="base_link" />
 			<child link="wheel_right_link" />
-			<origin xyz="0.0 ${-1*wheel_joint_y} ${wheel_joint_z}" rpy="0 0 ${M_PI}" />
+			<origin xyz="${wheel_joint_x} ${-1*wheel_joint_y} ${wheel_joint_z}" rpy="0 0 ${M_PI}" />
 			<axis xyz="0 -1 0" />
 		</joint>
@@ -242,5 +250,5 @@
 			<parent link="base_link" />
 			<child link="wheel_left_link" />
-			<origin xyz="0.0 ${wheel_joint_y} ${wheel_joint_z}" rpy="0 0 0" />
+			<origin xyz="${wheel_joint_x} ${wheel_joint_y} ${wheel_joint_z}" rpy="0 0 0" />
 			<axis xyz="0 1 0" />
 		</joint>
@@ -308,5 +316,4 @@
 			<minDepth>0</minDepth>
 			<maxVel>0.01</maxVel>
-			<fdir1>0 1 0</fdir1>
 			<material>Gazebo/Red</material>
 		</gazebo>
@@ -318,5 +325,4 @@
 			<minDepth>0</minDepth>
 			<maxVel>0.01</maxVel>
-			<fdir1>0 1 0</fdir1>
 			<material>Gazebo/Red</material>
 		</gazebo>
@@ -328,5 +334,4 @@
 			<minDepth>0</minDepth>
 			<maxVel>0.01</maxVel>
-			<fdir1>0 1 0</fdir1>
 			<material>Gazebo/Red</material>
 		</gazebo>
@@ -338,5 +343,4 @@
 			<minDepth>0</minDepth>
 			<maxVel>0.01</maxVel>
-			<fdir1>0 1 0</fdir1>
 			<material>Gazebo/Red</material>
 		</gazebo>
